Commit message: last night updates

File: body0.urdf (robot description, URDF)
Before this commit: robot robot, 5 links, 4 joints
Links:
- link Torso: geometry collision box size=0.7890828592531253 0.8464220222632227 0.6324885642457213; visual box size=0.7890828592531253 0.8464220222632227 0.6324885642457213
- link i0: geometry collision box size=0.40303704910125004 0.7104957598556476 0.2660532992342103; visual box size=0.40303704910125004 0.7104957598556476 0.2660532992342103
- link i1: geometry collision box size=0.24538272819719947 0.47830568227319636 0.3582141602980217; visual box size=0.24538272819719947 0.47830568227319636 0.3582141602980217
- link j0: geometry collision box size=0.9135356033232958 0.43421103049679666 0.5310433297612074; visual box size=0.9135356033232958 0.43421103049679666 0.5310433297612074
- link k0: geometry collision box size=0.8022305321814021 0.4134179295485527 0.44503170197787256; visual box size=0.8022305321814021 0.4134179295485527 0.44503170197787256
Joints:
- joint Torso_i0: origin xyz=0 0.4855524483815356 1.4833681682372262 rpy=0 0 1 -> xyz=0 0.42321101113161136 0.948732846368582 rpy=0 0 1
- joint Torso_j0: origin xyz=0 -0.4855524483815356 1.4833681682372262 rpy=0 0 1 -> xyz=0 -0.42321101113161136 0.948732846368582 rpy=0 0 1
- joint Torso_k0: origin xyz=0 0 1.9778242243163016 rpy=0 0 1 -> xyz=0 0 1.2649771284914426 rpy=0 0 1
- joint i0_i1: origin xyz=0 0.5340110595095544 0 rpy=1 0 0 -> xyz=0 0.7104957598556476 0 rpy=1 0 0

File: body1.urdf (robot description, URDF)
Before this commit: robot robot, 5 links, 4 joints
Links:
- link Torso: geometry collision box size=0.9521726609962777 0.6967517854483853 0.5366716248502328; visual box size=0.9521726609962777 0.6967517854483853 0.5366716248502328
- link i0: geometry collision box size=0.5039222914908552 0.6060733072567497 0.618806047715619; visual box size=0.5039222914908552 0.6060733072567497 0.618806047715619
- link i1: geometry collision box size=0.5901698705252084 0.9340227491636888 0.981951651073985; visual box size=0.5901698705252084 0.9340227491636888 0.981951651073985
- link j0: geometry collision box size=0.287540220432009 0.5690489177666624 0.33431927590945576; visual box size=0.287540220432009 0.5690489177666624 0.33431927590945576
- link k0: geometry collision box size=0.8333519269642444 0.5085141996427165 0.4687832677694395; visual box size=0.8333519269642444 0.5085141996427165 0.4687832677694395
Joints:
- joint Torso_i0: origin xyz=0 0.416478370650665 1.5765545035903052 rpy=1 0 0 -> xyz=0 0.34837589272419267 0.8050074372753492 rpy=0 0 1
- joint Torso_j0: origin xyz=0 -0.416478370650665 1.5765545035903052 rpy=0 0 1 -> xyz=0 -0.34837589272419267 0.8050074372753492 rpy=0 0 1
- joint Torso_k0: origin xyz=0 0 2.1020726714537403 rpy=0 0 1 -> xyz=0 0 1.0733432497004656 rpy=0 0 1
- joint i0_i1: origin xyz=0 0.5492283829312403 0 rpy=1 0 0 -> xyz=0 0.6060733072567497 0 rpy=1 0 0

File: body3.urdf (robot description, URDF)
Before this commit: robot robot, 5 links, 4 joints
Links:
- link Torso: geometry collision box size=0.9521726609962777 0.6967517854483853 0.5366716248502328; visual box size=0.9521726609962777 0.6967517854483853 0.5366716248502328
- link i0: geometry collision box size=0.5039222914908552 0.6060733072567497 0.618806047715619; visual box size=0.5039222914908552 0.6060733072567497 0.618806047715619
- link i1: geometry collision box size=0.5901698705252084 0.9340227491636888 0.981951651073985; visual box size=0.5901698705252084 0.9340227491636888 0.981951651073985
- link j0: geometry collision box size=0.287540220432009 0.5690489177666624 0.33431927590945576; visual box size=0.287540220432009 0.5690489177666624 0.33431927590945576
- link k0: geometry collision box size=0.8333519269642444 0.5085141996427165 0.4687832677694395; visual box size=0.8333519269642444 0.5085141996427165 0.4687832677694395
Joints:
- joint Torso_i0: origin xyz=0 0.416478370650665 1.5765545035903052 rpy=0 1 0 -> xyz=0 0.34837589272419267 0.8050074372753492 rpy=0 1 0
- joint Torso_j0: origin xyz=0 -0.416478370650665 1.5765545035903052 rpy=0 0 1 -> xyz=0 -0.34837589272419267 0.8050074372753492 rpy=0 0 1
- joint Torso_k0: origin xyz=0 0 2.1020726714537403 rpy=0 0 1 -> xyz=0 0 1.0733432497004656 rpy=0 0 1
- joint i0_i1: origin xyz=0 0.5492283829312403 0 rpy=1 0 0 -> xyz=0 0.6060733072567497 0 rpy=1 0 0

Commit message: cube, sensor, and joint names moved to __init__

File: body0.urdf (robot description, URDF)
Before this commit: robot robot, 5 links, 4 joints
Links:
- link Torso: geometry collision box size=0.7190346092943944 0.9500476929210759 0.6471387646528051; visual box size=0.7190346092943944 0.9500476929210759 0.6471387646528051
- link i0: geometry collision box size=0.4782622456487242 0.6495358669460073 0.6514740052333808; visual box size=0.4782622456487242 0.6495358669460073 0.6514740052333808
- link i1: geometry collision box size=0.8474229097432073 0.548898429243994 0.9241902187454165; visual box size=0.8474229097432073 0.548898429243994 0.9241902187454165
- link j0: geometry collision box size=0.5093080713163559 0.43364126740586767 0.43886797961304663; visual box size=0.5093080713163559 0.43364126740586767 0.43886797961304663
- link k0: geometry collision box size=0.4061914455532307 0.9484012803429744 0.545620677401391; visual box size=0.4061914455532307 0.9484012803429744 0.545620677401391
Joints:
- joint Torso_i0: origin xyz=0 0.42321101113161136 0.948732846368582 rpy=0 0 1 -> xyz=0 0.47502384646053797 0.9707081469792076 rpy=0 0 1
- joint Torso_j0: origin xyz=0 -0.42321101113161136 0.948732846368582 rpy=0 0 1 -> xyz=0 -0.47502384646053797 0.9707081469792076 rpy=0 0 1
- joint Torso_k0: origin xyz=0 0 1.2649771284914426 rpy=0 0 1 -> xyz=0 0 1.2942775293056101 rpy=0 0 1
- joint i0_i1: origin xyz=0 0.7104957598556476 0 rpy=1 0 0 -> xyz=0 0.6495358669460073 0 rpy=1 0 0

File: body1.urdf (robot description, URDF)
Before this commit: robot robot, 5 links, 4 joints
Links:
- link Torso: geometry collision box size=1.0472952589065423 0.5414331475600611 0.7701544422712611; visual box size=1.0472952589065423 0.5414331475600611 0.7701544422712611
- link i0: geometry collision box size=0.39393506075245627 0.9550607657471724 0.8963864876534904; visual box size=0.39393506075245627 0.9550607657471724 0.8963864876534904
- link i1: geometry collision box size=0.35045192724085167 0.32260869832076555 0.7963501312790024; visual box size=0.35045192724085167 0.32260869832076555 0.7963501312790024
- link j0: geometry collision box size=0.48096108039598884 0.4019854325021977 0.36635534819304055; visual box size=0.48096108039598884 0.4019854325021977 0.36635534819304055
- link k0: geometry collision box size=0.4638232838589687 0.7222471802600261 0.5492444082073253; visual box size=0.4638232838589687 0.7222471802600261 0.5492444082073253
Joints:
- joint Torso_i0: origin xyz=0 0.34837589272419267 0.8050074372753492 rpy=0 0 1 -> xyz=0 0.27071657378003056 1.1552316634068915 rpy=1 0 0
- joint Torso_j0: origin xyz=0 -0.34837589272419267 0.8050074372753492 rpy=0 0 1 -> xyz=0 -0.27071657378003056 1.1552316634068915 rpy=0 0 1
- joint Torso_k0: origin xyz=0 0 1.0733432497004656 rpy=0 0 1 -> xyz=0 0 1.5403088845425221 rpy=0 0 1
- joint i0_i1: origin xyz=0 0.6060733072567497 0 rpy=1 0 0 -> xyz=0 0.9550607657471724 0 rpy=1 0 0

File: body3.urdf (robot description, URDF)
Before this commit: robot robot, 5 links, 4 joints
Links:
- link Torso: geometry collision box size=1.0472952589065423 0.5414331475600611 0.7701544422712611; visual box size=1.0472952589065423 0.5414331475600611 0.7701544422712611
- link i0: geometry collision box size=0.39393506075245627 0.9550607657471724 0.8963864876534904; visual box size=0.39393506075245627 0.9550607657471724 0.8963864876534904
- link i1: geometry collision box size=0.35045192724085167 0.32260869832076555 0.7963501312790024; visual box size=0.35045192724085167 0.32260869832076555 0.7963501312790024
- link j0: geometry collision box size=0.48096108039598884 0.4019854325021977 0.36635534819304055; visual box size=0.48096108039598884 0.4019854325021977 0.36635534819304055
- link k0: geometry collision box size=0.4638232838589687 0.7222471802600261 0.5492444082073253; visual box size=0.4638232838589687 0.7222471802600261 0.5492444082073253
Joints:
- joint Torso_i0: origin xyz=0 0.34837589272419267 0.8050074372753492 rpy=0 1 0 -> xyz=0 0.27071657378003056 1.1552316634068915 rpy=0 0 1
- joint Torso_j0: origin xyz=0 -0.34837589272419267 0.8050074372753492 rpy=0 0 1 -> xyz=0 -0.27071657378003056 1.1552316634068915 rpy=0 0 1
- joint Torso_k0: origin xyz=0 0 1.0733432497004656 rpy=0 0 1 -> xyz=0 0 1.5403088845425221 rpy=0 0 1
- joint i0_i1: origin xyz=0 0.6060733072567497 0 rpy=1 0 0 -> xyz=0 0.9550607657471724 0 rpy=1 0 0

Commit message: synapse loop is iterating a billion times???

File: body0.urdf (robot description, URDF)
Before this commit: robot robot, 5 links, 4 joints
Links:
- added link j1, mass 1; collision box size=0.23348546910026935 0.2594215194291839 0.9410737100217683; visual box size=0.23348546910026935 0.2594215194291839 0.9410737100217683
- added link k1, mass 1; collision box size=0.4338664277024372 0.22044730057157225 0.8602863544982438; visual box size=0.4338664277024372 0.22044730057157225 0.8602863544982438
- link Torso: geometry collision box size=0.621191207697974 0.7527295983736758 1.0337139480541597; visual box size=0.621191207697974 0.7527295983736758 1.0337139480541597
- link i0: geometry collision box size=0.6217852083178159 0.810214500140644 0.962029956129612; visual box size=0.6217852083178159 0.810214500140644 0.962029956129612
- link i1: geometry collision box size=0.3763225095384611 0.26449766726951557 0.6284532779206626; visual box size=0.3763225095384611 0.26449766726951557 0.6284532779206626
- link j0: geometry collision box size=0.6968783483305947 0.3848403408449798 0.6005423275555427; visual box size=0.6968783483305947 0.3848403408449798 0.6005423275555427
- link k0: geometry collision box size=0.23948321404719064 0.9987530132489535 0.7288010782652139; visual box size=0.23948321404719064 0.9987530132489535 0.7288010782652139
Joints:
- added joint j0_j1: type revolute, parent j0, child j1, origin xyz=0 -0.3848403408449798 0 rpy=1 0 0, axis 1 0 0, limit lower=-3.14159 upper=3.14159 effort=0.0 velocity=0.0
- added joint k0_k1: type revolute, parent k0, child k1, origin xyz=0 0 0.7288010782652139 rpy=1 0 0, axis 1 0 0, limit lower=-3.14159 upper=3.14159 effort=0.0 velocity=0.0
- joint Torso_i0: origin xyz=0 0.47502384646053797 0.9707081469792076 rpy=0 0 1 -> xyz=0 0.3763647991868379 1.5505709220812396 rpy=0 0 1
- joint Torso_j0: origin xyz=0 -0.47502384646053797 0.9707081469792076 rpy=0 0 1 -> xyz=0 -0.3763647991868379 1.5505709220812396 rpy=0 0 1
- joint Torso_k0: origin xyz=0 0 1.2942775293056101 rpy=0 0 1 -> xyz=0 0 2.0674278961083195 rpy=0 0 1
- joint i0_i1: origin xyz=0 0.6495358669460073 0 rpy=1 0 0 -> xyz=0 0.810214500140644 0 rpy=1 0 0

File: body1.urdf (robot description, URDF)
Before this commit: robot robot, 5 links, 4 joints
Links:
- added link j1, mass 1; collision box size=0.7630892131067748 0.9813223782993368 0.9740628467059147; visual box size=0.7630892131067748 0.9813223782993368 0.9740628467059147
- added link k1, mass 1; collision box size=0.9169916798508682 0.28009581778659814 0.5825400321624075; visual box size=0.9169916798508682 0.28009581778659814 0.5825400321624075
- link Torso: geometry collision box size=0.5608220265967023 0.4548734478187786 0.5564510991682344; visual box size=0.5608220265967023 0.4548734478187786 0.5564510991682344
- link i0: geometry collision box size=0.3333131743519916 0.2716516156308405 0.8083993902269186; visual box size=0.3333131743519916 0.2716516156308405 0.8083993902269186
- link i1: geometry collision box size=0.9623411497225596 0.35474764967380373 0.21589386052588255; visual box size=0.9623411497225596 0.35474764967380373 0.21589386052588255
- link j0: geometry collision box size=0.3246977394216837 0.6757269317208682 0.37661617106514095; visual box size=0.3246977394216837 0.6757269317208682 0.37661617106514095
- link k0: geometry collision box size=0.8835322411586584 0.9031588048872556 0.5808244923139367; visual box size=0.8835322411586584 0.9031588048872556 0.5808244923139367
Joints:
- added joint j0_j1: type revolute, parent j0, child j1, origin xyz=0 -0.6757269317208682 0 rpy=1 0 0, axis 1 0 0, limit lower=-3.14159 upper=3.14159 effort=0.0 velocity=0.0
- added joint k0_k1: type revolute, parent k0, child k1, origin xyz=0 0 0.5808244923139367 rpy=1 0 0, axis 1 0 0, limit lower=-3.14159 upper=3.14159 effort=0.0 velocity=0.0
- joint Torso_i0: origin xyz=0 0.27071657378003056 1.1552316634068915 rpy=1 0 0 -> xyz=0 0.2274367239093893 0.8346766487523516 rpy=0 0 1
- joint Torso_j0: origin xyz=0 -0.27071657378003056 1.1552316634068915 rpy=0 0 1 -> xyz=0 -0.2274367239093893 0.8346766487523516 rpy=0 0 1
- joint Torso_k0: origin xyz=0 0 1.5403088845425221 rpy=0 0 1 -> xyz=0 0 1.1129021983364689 rpy=0 0 1
- joint i0_i1: origin xyz=0 0.9550607657471724 0 rpy=1 0 0 -> xyz=0 0.2716516156308405 0 rpy=1 0 0

File: body2.urdf (robot description, URDF)
Before this commit: robot robot, 5 links, 4 joints
Links:
- added link j1, mass 1; collision box size=0.35667362814158904 0.7396858521927496 0.6900674850506239; visual box size=0.35667362814158904 0.7396858521927496 0.6900674850506239
- added link k1, mass 1; collision box size=0.8945247223455517 0.7586330118535183 0.23226897273533542; visual box size=0.8945247223455517 0.7586330118535183 0.23226897273533542
- link Torso: geometry collision box size=0.8879728456884713 0.5160897149413571 0.9088638372105096; visual box size=0.8879728456884713 0.5160897149413571 0.9088638372105096
- link i0: geometry collision box size=0.3855454426386543 0.27981105687016206 0.5045402513397115; visual box size=0.3855454426386543 0.27981105687016206 0.5045402513397115
- link i1: geometry collision box size=0.9569557527737957 0.825725389581047 0.9711271272171917; visual box size=0.9569557527737957 0.825725389581047 0.9711271272171917
- link j0: geometry collision box size=0.7366108940529765 0.6935352544354747 0.5070276518162067; visual box size=0.7366108940529765 0.6935352544354747 0.5070276518162067
- link k0: geometry collision box size=0.27349857741988615 0.9356937163124177 0.4939403717761522; visual box size=0.27349857741988615 0.9356937163124177 0.4939403717761522
Joints:
- added joint j0_j1: type revolute, parent j0, child j1, origin xyz=0 -0.6935352544354747 0 rpy=1 0 0, axis 1 0 0, limit lower=-3.14159 upper=3.14159 effort=0.0 velocity=0.0
- added joint k0_k1: type revolute, parent k0, child k1, origin xyz=0 0 0.4939403717761522 rpy=1 0 0, axis 1 0 0, limit lower=-3.14159 upper=3.14159 effort=0.0 velocity=0.0
- joint Torso_i0: origin xyz=0 0.47502384646053797 0.9707081469792076 rpy=0 0 1 -> xyz=0 0.25804485747067857 1.3632957558157643 rpy=0 0 0
- joint Torso_j0: origin xyz=0 -0.47502384646053797 0.9707081469792076 rpy=0 0 1 -> xyz=0 -0.25804485747067857 1.3632957558157643 rpy=0 0 1
- joint Torso_k0: origin xyz=0 0 1.2942775293056101 rpy=0 0 1 -> xyz=0 0 1.8177276744210191 rpy=0 0 1
- joint i0_i1: origin xyz=0 0.6495358669460073 0 rpy=1 0 0 -> xyz=0 0.27981105687016206 0 rpy=1 0 0

File: body3.urdf (robot description, URDF)
Before this commit: robot robot, 5 links, 4 joints
Links:
- added link j1, mass 1; collision box size=0.39402517031047035 0.3628973163984288 0.9119109539994976; visual box size=0.39402517031047035 0.3628973163984288 0.9119109539994976
- added link k1, mass 1; collision box size=0.3427619155778464 0.2808294692595692 0.5405972237351115; visual box size=0.3427619155778464 0.2808294692595692 0.5405972237351115
- link Torso: geometry collision box size=1.0296231097449347 0.5293628277013105 0.5974381220017878; visual box size=1.0296231097449347 0.5293628277013105 0.5974381220017878
- link i0: geometry collision box size=0.9441661004037984 0.2655590130441951 0.9214408631013211; visual box size=0.9441661004037984 0.2655590130441951 0.9214408631013211
- link i1: geometry collision box size=0.23497511386813646 0.47301964679547237 0.615767981817865; visual box size=0.23497511386813646 0.47301964679547237 0.615767981817865
- link j0: geometry collision box size=0.6777872065446533 0.6522729637207352 0.4930014970869486; visual box size=0.6777872065446533 0.6522729637207352 0.4930014970869486
- link k0: geometry collision box size=0.5548294535553333 0.5159935158569909 0.7189718147597957; visual box size=0.5548294535553333 0.5159935158569909 0.7189718147597957
Joints:
- added joint j0_j1: type revolute, parent j0, child j1, origin xyz=0 -0.6522729637207352 0 rpy=1 0 0, axis 1 0 0, limit lower=-3.14159 upper=3.14159 effort=0.0 velocity=0.0
- added joint k0_k1: type revolute, parent k0, child k1, origin xyz=0 0 0.7189718147597957 rpy=1 0 0, axis 1 0 0, limit lower=-3.14159 upper=3.14159 effort=0.0 velocity=0.0
- joint Torso_i0: origin xyz=0 0.27071657378003056 1.1552316634068915 rpy=0 0 1 -> xyz=0 0.26468141385065524 0.8961571830026818 rpy=0 1 0
- joint Torso_j0: origin xyz=0 -0.27071657378003056 1.1552316634068915 rpy=0 0 1 -> xyz=0 -0.26468141385065524 0.8961571830026818 rpy=0 0 1
- joint Torso_k0: origin xyz=0 0 1.5403088845425221 rpy=0 0 1 -> xyz=0 0 1.1948762440035756 rpy=0 0 1
- joint i0_i1: origin xyz=0 0.9550607657471724 0 rpy=1 0 0 -> xyz=0 0.2655590130441951 0 rpy=1 0 0
