Commit message: synapses working, refine mutate()

File: body0.urdf (robot description, URDF)
Before this commit: robot robot, 7 links, 6 joints
Links:
- link Torso: geometry collision box size=0.7457217872955 1.2391614648796434 1.018665655562691; visual box size=0.7457217872955 1.2391614648796434 1.018665655562691
- link i0: geometry collision box size=0.3647805613091107 0.9898086850351462 0.9426492066878431; visual box size=0.3647805613091107 0.9898086850351462 0.9426492066878431
- link i1: geometry collision box size=0.8358903922505487 0.7114324900959741 0.5803050675607425; visual box size=0.8358903922505487 0.7114324900959741 0.5803050675607425
- link j0: geometry collision box size=0.734106859332893 0.27224610714888436 0.39351845931919416; visual box size=0.734106859332893 0.27224610714888436 0.39351845931919416
- link j1: geometry collision box size=0.3343743004995835 0.9684706052379202 0.3592385575145658; visual box size=0.3343743004995835 0.9684706052379202 0.3592385575145658
- link k0: geometry collision box size=0.7816771161580787 0.40845501031137604 0.5321029169218512; visual box size=0.7816771161580787 0.40845501031137604 0.5321029169218512
- link k1: geometry collision box size=0.2519735754867311 0.8627079957208761 0.28877601140244424; visual box size=0.2519735754867311 0.8627079957208761 0.28877601140244424
Joints:
- joint Torso_i0: origin xyz=0 0.3763647991868379 1.5505709220812396 rpy=0 0 1 -> xyz=0 0.6195807324398217 1.5279984833440365 rpy=0 1 0
- joint Torso_j0: origin xyz=0 -0.3763647991868379 1.5505709220812396 rpy=0 0 1 -> xyz=0 -0.6195807324398217 1.5279984833440365 rpy=0 0 1
- joint Torso_k0: origin xyz=0 0 2.0674278961083195 rpy=0 0 1 -> xyz=0 0 2.037331311125382 rpy=0 0 1
- joint i0_i1: origin xyz=0 0.810214500140644 0 rpy=1 0 0 -> xyz=0 0.9898086850351462 0 rpy=1 0 0
- joint j0_j1: origin xyz=0 -0.3848403408449798 0 rpy=1 0 0 -> xyz=0 -0.27224610714888436 0 rpy=1 0 0
- joint k0_k1: origin xyz=0 0 0.7288010782652139 rpy=1 0 0 -> xyz=0 0 0.5321029169218512 rpy=1 0 0

File: body1.urdf (robot description, URDF)
Before this commit: robot robot, 7 links, 6 joints
Links:
- link Torso: geometry collision box size=0.7457217872955 1.2391614648796434 1.018665655562691; visual box size=0.7457217872955 1.2391614648796434 1.018665655562691
- link i0: geometry collision box size=0.3647805613091107 0.9898086850351462 0.9426492066878431; visual box size=0.3647805613091107 0.9898086850351462 0.9426492066878431
- link i1: geometry collision box size=0.8358903922505487 0.7114324900959741 0.5803050675607425; visual box size=0.8358903922505487 0.7114324900959741 0.5803050675607425
- link j0: geometry collision box size=0.734106859332893 0.27224610714888436 0.39351845931919416; visual box size=0.734106859332893 0.27224610714888436 0.39351845931919416
- link j1: geometry collision box size=0.3343743004995835 0.9684706052379202 0.3592385575145658; visual box size=0.3343743004995835 0.9684706052379202 0.3592385575145658
- link k0: geometry collision box size=0.7816771161580787 0.40845501031137604 0.5321029169218512; visual box size=0.7816771161580787 0.40845501031137604 0.5321029169218512
- link k1: geometry collision box size=0.2519735754867311 0.8627079957208761 0.28877601140244424; visual box size=0.2519735754867311 0.8627079957208761 0.28877601140244424
Joints:
- joint Torso_i0: origin xyz=0 0.2274367239093893 0.8346766487523516 rpy=0 0 1 -> xyz=0 0.6195807324398217 1.5279984833440365 rpy=0 0 0
- joint Torso_j0: origin xyz=0 -0.2274367239093893 0.8346766487523516 rpy=0 0 1 -> xyz=0 -0.6195807324398217 1.5279984833440365 rpy=0 0 1
- joint Torso_k0: origin xyz=0 0 1.1129021983364689 rpy=0 0 1 -> xyz=0 0 2.037331311125382 rpy=0 0 1
- joint i0_i1: origin xyz=0 0.2716516156308405 0 rpy=1 0 0 -> xyz=0 0.9898086850351462 0 rpy=1 0 0
- joint j0_j1: origin xyz=0 -0.6757269317208682 0 rpy=1 0 0 -> xyz=0 -0.27224610714888436 0 rpy=1 0 0
- joint k0_k1: origin xyz=0 0 0.5808244923139367 rpy=1 0 0 -> xyz=0 0 0.5321029169218512 rpy=1 0 0

File: body2.urdf (robot description, URDF)
Before this commit: robot robot, 7 links, 6 joints
Links:
- link Torso: geometry collision box size=0.7457217872955 1.2391614648796434 1.018665655562691; visual box size=0.7457217872955 1.2391614648796434 1.018665655562691
- link i0: geometry collision box size=0.3647805613091107 0.9898086850351462 0.9426492066878431; visual box size=0.3647805613091107 0.9898086850351462 0.9426492066878431
- link i1: geometry collision box size=0.8358903922505487 0.7114324900959741 0.5803050675607425; visual box size=0.8358903922505487 0.7114324900959741 0.5803050675607425
- link j0: geometry collision box size=0.734106859332893 0.27224610714888436 0.39351845931919416; visual box size=0.734106859332893 0.27224610714888436 0.39351845931919416
- link j1: geometry collision box size=0.3343743004995835 0.9684706052379202 0.3592385575145658; visual box size=0.3343743004995835 0.9684706052379202 0.3592385575145658
- link k0: geometry collision box size=0.7816771161580787 0.40845501031137604 0.5321029169218512; visual box size=0.7816771161580787 0.40845501031137604 0.5321029169218512
- link k1: geometry collision box size=0.2519735754867311 0.8627079957208761 0.28877601140244424; visual box size=0.2519735754867311 0.8627079957208761 0.28877601140244424
Joints:
- joint Torso_i0: origin xyz=0 0.25804485747067857 1.3632957558157643 rpy=0 0 0 -> xyz=0 0.6195807324398217 1.5279984833440365 rpy=0 1 0
- joint Torso_j0: origin xyz=0 -0.25804485747067857 1.3632957558157643 rpy=0 0 1 -> xyz=0 -0.6195807324398217 1.5279984833440365 rpy=0 0 1
- joint Torso_k0: origin xyz=0 0 1.8177276744210191 rpy=0 0 1 -> xyz=0 0 2.037331311125382 rpy=0 0 1
- joint i0_i1: origin xyz=0 0.27981105687016206 0 rpy=1 0 0 -> xyz=0 0.9898086850351462 0 rpy=1 0 0
- joint j0_j1: origin xyz=0 -0.6935352544354747 0 rpy=1 0 0 -> xyz=0 -0.27224610714888436 0 rpy=1 0 0
- joint k0_k1: origin xyz=0 0 0.4939403717761522 rpy=1 0 0 -> xyz=0 0 0.5321029169218512 rpy=1 0 0

File: body3.urdf (robot description, URDF)
Before this commit: robot robot, 7 links, 6 joints
Links:
- link Torso: geometry collision box size=0.7457217872955 1.2391614648796434 1.018665655562691; visual box size=0.7457217872955 1.2391614648796434 1.018665655562691
- link i0: geometry collision box size=0.3647805613091107 0.9898086850351462 0.9426492066878431; visual box size=0.3647805613091107 0.9898086850351462 0.9426492066878431
- link i1: geometry collision box size=0.8358903922505487 0.7114324900959741 0.5803050675607425; visual box size=0.8358903922505487 0.7114324900959741 0.5803050675607425
- link j0: geometry collision box size=0.734106859332893 0.27224610714888436 0.39351845931919416; visual box size=0.734106859332893 0.27224610714888436 0.39351845931919416
- link j1: geometry collision box size=0.3343743004995835 0.9684706052379202 0.3592385575145658; visual box size=0.3343743004995835 0.9684706052379202 0.3592385575145658
- link k0: geometry collision box size=0.7816771161580787 0.40845501031137604 0.5321029169218512; visual box size=0.7816771161580787 0.40845501031137604 0.5321029169218512
- link k1: geometry collision box size=0.2519735754867311 0.8627079957208761 0.28877601140244424; visual box size=0.2519735754867311 0.8627079957208761 0.28877601140244424
Joints:
- joint Torso_i0: origin xyz=0 0.26468141385065524 0.8961571830026818 rpy=0 1 0 -> xyz=0 0.6195807324398217 1.5279984833440365 rpy=0 0 0
- joint Torso_j0: origin xyz=0 -0.26468141385065524 0.8961571830026818 rpy=0 0 1 -> xyz=0 -0.6195807324398217 1.5279984833440365 rpy=0 0 1
- joint Torso_k0: origin xyz=0 0 1.1948762440035756 rpy=0 0 1 -> xyz=0 0 2.037331311125382 rpy=0 0 1
- joint i0_i1: origin xyz=0 0.2655590130441951 0 rpy=1 0 0 -> xyz=0 0.9898086850351462 0 rpy=1 0 0
- joint j0_j1: origin xyz=0 -0.6522729637207352 0 rpy=1 0 0 -> xyz=0 -0.27224610714888436 0 rpy=1 0 0
- joint k0_k1: origin xyz=0 0 0.7189718147597957 rpy=1 0 0 -> xyz=0 0 0.5321029169218512 rpy=1 0 0

File: body4.urdf (robot description, URDF)
Before this commit: robot robot, 7 links, 6 joints
Links:
- link Torso: geometry collision box size=0.7457217872955 1.2391614648796434 1.018665655562691; visual box size=0.7457217872955 1.2391614648796434 1.018665655562691
- link i0: geometry collision box size=0.3647805613091107 0.9898086850351462 0.9426492066878431; visual box size=0.3647805613091107 0.9898086850351462 0.9426492066878431
- link i1: geometry collision box size=0.8358903922505487 0.7114324900959741 0.5803050675607425; visual box size=0.8358903922505487 0.7114324900959741 0.5803050675607425
- link j0: geometry collision box size=0.734106859332893 0.27224610714888436 0.39351845931919416; visual box size=0.734106859332893 0.27224610714888436 0.39351845931919416
- link j1: geometry collision box size=0.3343743004995835 0.9684706052379202 0.3592385575145658; visual box size=0.3343743004995835 0.9684706052379202 0.3592385575145658
- link k0: geometry collision box size=0.7816771161580787 0.40845501031137604 0.5321029169218512; visual box size=0.7816771161580787 0.40845501031137604 0.5321029169218512
- link k1: geometry collision box size=0.2519735754867311 0.8627079957208761 0.28877601140244424; visual box size=0.2519735754867311 0.8627079957208761 0.28877601140244424
Joints:
- joint Torso_i0: origin xyz=0 0.20037864348178183 0.7478645451311896 rpy=0 0 0 -> xyz=0 0.6195807324398217 1.5279984833440365 rpy=0 0 1
- joint Torso_j0: origin xyz=0 -0.20037864348178183 0.7478645451311896 rpy=0 0 1 -> xyz=0 -0.6195807324398217 1.5279984833440365 rpy=0 0 1
- joint Torso_k0: origin xyz=0 0 0.9971527268415861 rpy=0 0 1 -> xyz=0 0 2.037331311125382 rpy=0 0 1
- joint i0_i1: origin xyz=0 0.8716075415561872 0 rpy=1 0 0 -> xyz=0 0.9898086850351462 0 rpy=1 0 0
- joint j0_j1: origin xyz=0 -0.23469806982327254 0 rpy=1 0 0 -> xyz=0 -0.27224610714888436 0 rpy=1 0 0
- joint k0_k1: origin xyz=0 0 0.8997889133233428 rpy=1 0 0 -> xyz=0 0 0.5321029169218512 rpy=1 0 0

File: body5.urdf (robot description, URDF)
Before this commit: robot robot, 7 links, 6 joints
Links:
- link Torso: geometry collision box size=0.7457217872955 1.2391614648796434 1.018665655562691; visual box size=0.7457217872955 1.2391614648796434 1.018665655562691
- link i0: geometry collision box size=0.3647805613091107 0.9898086850351462 0.9426492066878431; visual box size=0.3647805613091107 0.9898086850351462 0.9426492066878431
- link i1: geometry collision box size=0.8358903922505487 0.7114324900959741 0.5803050675607425; visual box size=0.8358903922505487 0.7114324900959741 0.5803050675607425
- link j0: geometry collision box size=0.734106859332893 0.27224610714888436 0.39351845931919416; visual box size=0.734106859332893 0.27224610714888436 0.39351845931919416
- link j1: geometry collision box size=0.3343743004995835 0.9684706052379202 0.3592385575145658; visual box size=0.3343743004995835 0.9684706052379202 0.3592385575145658
- link k0: geometry collision box size=0.7816771161580787 0.40845501031137604 0.5321029169218512; visual box size=0.7816771161580787 0.40845501031137604 0.5321029169218512
- link k1: geometry collision box size=0.2519735754867311 0.8627079957208761 0.28877601140244424; visual box size=0.2519735754867311 0.8627079957208761 0.28877601140244424
Joints:
- joint Torso_i0: origin xyz=0 0.27199916975127636 1.4677012067060229 rpy=0 1 0 -> xyz=0 0.6195807324398217 1.5279984833440365 rpy=1 0 0
- joint Torso_j0: origin xyz=0 -0.27199916975127636 1.4677012067060229 rpy=0 0 1 -> xyz=0 -0.6195807324398217 1.5279984833440365 rpy=0 0 1
- joint Torso_k0: origin xyz=0 0 1.956934942274697 rpy=0 0 1 -> xyz=0 0 2.037331311125382 rpy=0 0 1
- joint i0_i1: origin xyz=0 0.8839810179758241 0 rpy=1 0 0 -> xyz=0 0.9898086850351462 0 rpy=1 0 0
- joint j0_j1: origin xyz=0 -0.2650888950612032 0 rpy=1 0 0 -> xyz=0 -0.27224610714888436 0 rpy=1 0 0
- joint k0_k1: origin xyz=0 0 0.3269272429533231 rpy=1 0 0 -> xyz=0 0 0.5321029169218512 rpy=1 0 0

File: body6.urdf (robot description, URDF)
Before this commit: robot robot, 7 links, 6 joints
Links:
- removed link k1
- added link i2, mass 1; collision box size=0.7451641194843992 0.9857019846905177 0.9381075909805321; visual box size=0.7451641194843992 0.9857019846905177 0.9381075909805321
- added link j2, mass 1; collision box size=0.3219117008061358 0.5204671986245843 0.7528249234357138; visual box size=0.3219117008061358 0.5204671986245843 0.7528249234357138
- link Torso: geometry collision box size=0.46167313819334416 0.7502481053079376 0.4645817551633846; visual box size=0.46167313819334416 0.7502481053079376 0.4645817551633846
- link i0: geometry collision box size=0.7961146295254509 0.6362546528634063 0.30193759425128297; visual box size=0.7961146295254509 0.6362546528634063 0.30193759425128297
- link i1: geometry collision box size=0.2654814939308778 0.3508762899364235 0.33733332873224536; visual box size=0.2654814939308778 0.3508762899364235 0.33733332873224536
- link j0: geometry collision box size=0.3628207699297645 0.5195416040203034 0.3099975738147793; visual box size=0.3628207699297645 0.5195416040203034 0.3099975738147793
- link j1: geometry collision box size=0.23779201457095206 0.20597220288945162 0.4416340967568262; visual box size=0.23779201457095206 0.20597220288945162 0.4416340967568262
- link k0: geometry collision box size=0.6005768596982344 0.5645138426197844 0.825431706306557; visual box size=0.6005768596982344 0.5645138426197844 0.825431706306557
Joints:
- removed joint k0_k1
- added joint i1_i2: type revolute, parent i1, child i2, origin xyz=0 0.3508762899364235 0 rpy=1 0 0, axis 1 0 0, limit lower=-3.14159 upper=3.14159 effort=0.0 velocity=0.0
- added joint j1_j2: type revolute, parent j1, child j2, origin xyz=0 -0.20597220288945162 0 rpy=1 0 0, axis 1 0 0, limit lower=-3.14159 upper=3.14159 effort=0.0 velocity=0.0
- joint Torso_i0: origin xyz=0 0.5176119385933335 1.439310943912083 rpy=0 0 1 -> xyz=0 0.3751240526539688 0.6968726327450769 rpy=1 0 0
- joint Torso_j0: origin xyz=0 -0.5176119385933335 1.439310943912083 rpy=0 0 1 -> xyz=0 -0.3751240526539688 0.6968726327450769 rpy=0 0 1
- joint Torso_k0: origin xyz=0 0 1.919081258549444 rpy=0 0 1 -> xyz=0 0 0.9291635103267692 rpy=0 0 1
- joint i0_i1: origin xyz=0 0.24110203575562927 0 rpy=1 0 0 -> xyz=0 0.6362546528634063 0 rpy=1 0 0
- joint j0_j1: origin xyz=0 -0.6067359602266038 0 rpy=1 0 0 -> xyz=0 -0.5195416040203034 0 rpy=1 0 0

File: body7.urdf (robot description, URDF)
Before this commit: robot robot, 7 links, 6 joints
Links:
- removed link i1
- link Torso: geometry collision box size=0.621641728329736 0.6407264316567994 0.8867551054785079; visual box size=0.621641728329736 0.6407264316567994 0.8867551054785079
- link i0: geometry collision box size=0.26852160096233385 0.9856943330997818 0.5798798259279325; visual box size=0.26852160096233385 0.9856943330997818 0.5798798259279325
- link j0: geometry collision box size=0.7832798477954126 0.8201764700925045 0.5261341035915805; visual box size=0.7832798477954126 0.8201764700925045 0.5261341035915805
- link j1: geometry collision box size=0.42205254724789126 0.5584825224888563 0.3957656095269704; visual box size=0.42205254724789126 0.5584825224888563 0.3957656095269704
- link k0: geometry collision box size=0.8557194405073614 0.6917749888939406 0.4564969888340068; visual box size=0.8557194405073614 0.6917749888939406 0.4564969888340068
- link k1: geometry collision box size=0.4997835102674712 0.36851296216301865 0.6131648379547752; visual box size=0.4997835102674712 0.36851296216301865 0.6131648379547752
Joints:
- removed joint i0_i1
- joint Torso_i0: origin xyz=0 0.4850071085361873 1.5920629107503064 rpy=0 0 1 -> xyz=0 0.3203632158283997 1.330132658217762 rpy=0 1 0
- joint Torso_j0: origin xyz=0 -0.4850071085361873 1.5920629107503064 rpy=0 0 1 -> xyz=0 -0.3203632158283997 1.330132658217762 rpy=0 0 1
- joint Torso_k0: origin xyz=0 0 2.122750547667075 rpy=0 0 1 -> xyz=0 0 1.7735102109570158 rpy=0 0 1
- joint j0_j1: origin xyz=0 -0.5451719322939499 0 rpy=1 0 0 -> xyz=0 -0.8201764700925045 0 rpy=1 0 0
- joint k0_k1: origin xyz=0 0 0.6536996777850941 rpy=1 0 0 -> xyz=0 0 0.4564969888340068 rpy=1 0 0

File: body8.urdf (robot description, URDF)
Before this commit: robot robot, 7 links, 6 joints
Links:
- removed link i1
- removed link j0
- removed link j1
- removed link k0
- removed link k1
- link Torso: geometry collision box size=0.7894706267661382 0.43538243131952775 0.4098540367859649; visual box size=0.7894706267661382 0.43538243131952775 0.4098540367859649
- link i0: geometry collision box size=0.6931558611961564 0.2566280006727933 0.7375405665439676; visual box size=0.6931558611961564 0.2566280006727933 0.7375405665439676
Joints:
- removed joint Torso_j0
- removed joint Torso_k0
- removed joint i0_i1
- removed joint j0_j1
- removed joint k0_k1
- joint Torso_i0: origin xyz=0 0.611191258508751 1.5212748466174975 rpy=0 1 0 -> xyz=0 0.21769121565976388 0.6147810551789473 rpy=0 1 0

File: body9.urdf (robot description, URDF)
Before this commit: robot robot, 7 links, 6 joints
Links:
- removed link j0
- removed link j1
- removed link k1
- added link i2, mass 1; collision box size=0.22471520475591494 0.8362233786791942 0.827981830801874; visual box size=0.22471520475591494 0.8362233786791942 0.827981830801874
- link Torso: geometry collision box size=1.2560077824879863 0.7626164383225629 0.4635933424436314; visual box size=1.2560077824879863 0.7626164383225629 0.4635933424436314
- link i0: geometry collision box size=0.9038417127411651 0.3015601719956716 0.7040499786211938; visual box size=0.9038417127411651 0.3015601719956716 0.7040499786211938
- link i1: geometry collision box size=0.3142895449277962 0.7995191416822478 0.457063238737286; visual box size=0.3142895449277962 0.7995191416822478 0.457063238737286
- link k0: geometry collision box size=0.7755604621490846 0.20024793083323056 0.2864631606978851; visual box size=0.7755604621490846 0.20024793083323056 0.2864631606978851
Joints:
- removed joint Torso_j0
- removed joint j0_j1
- removed joint k0_k1
- added joint i1_i2: type revolute, parent i1, child i2, origin xyz=0 0.7995191416822478 0 rpy=1 0 0, axis 1 0 0, limit lower=-3.14159 upper=3.14159 effort=0.0 velocity=0.0
- joint Torso_i0: origin xyz=0 0.4036149103685446 1.2359697168014252 rpy=0 0 0 -> xyz=0 0.38130821916128144 0.6953900136654471 rpy=0 1 0
- joint Torso_k0: origin xyz=0 0 1.6479596224019004 rpy=0 0 1 -> xyz=0 0 0.9271866848872627 rpy=0 0 1
- joint i0_i1: origin xyz=0 0.9609116589203626 0 rpy=1 0 0 -> xyz=0 0.3015601719956716 0 rpy=1 0 0
