Commit message: synapses working, refine mutate()

File: body0.urdf (robot description, URDF)
Before this commit: robot robot, 7 links, 6 joints
Links:
- link Torso: geometry collision box size=0.4270820660990066 1.0538899660439736 1.152347599706828; visual box size=0.4270820660990066 1.0538899660439736 1.152347599706828
- link i0: geometry collision box size=0.4662786948372766 0.20670083978720682 0.24069037165999171; visual box size=0.4662786948372766 0.20670083978720682 0.24069037165999171
- link i1: geometry collision box size=0.42713318362025565 0.9490551511654679 0.6150144779125608; visual box size=0.42713318362025565 0.9490551511654679 0.6150144779125608
- link j0: geometry collision box size=0.3508349298730473 0.23362430842753437 0.8934338651499589; visual box size=0.3508349298730473 0.23362430842753437 0.8934338651499589
- link j1: geometry collision box size=0.847778629833061 0.6659606540101592 0.9166403317259235; visual box size=0.847778629833061 0.6659606540101592 0.9166403317259235
- link k0: geometry collision box size=0.6140921707159852 0.6159897364099624 0.8581481960782829; visual box size=0.6140921707159852 0.6159897364099624 0.8581481960782829
- link k1: geometry collision box size=0.8083844113766532 0.7965283546037021 0.814354034299329; visual box size=0.8083844113766532 0.7965283546037021 0.814354034299329
Joints:
- joint Torso_i0: origin xyz=0 0.6195807324398217 1.5279984833440365 rpy=0 1 0 -> xyz=0 0.5269449830219868 1.728521399560242 rpy=1 0 0
- joint Torso_j0: origin xyz=0 -0.6195807324398217 1.5279984833440365 rpy=0 0 1 -> xyz=0 -0.5269449830219868 1.728521399560242 rpy=0 0 1
- joint Torso_k0: origin xyz=0 0 2.037331311125382 rpy=0 0 1 -> xyz=0 0 2.304695199413656 rpy=0 0 1
- joint i0_i1: origin xyz=0 0.9898086850351462 0 rpy=1 0 0 -> xyz=0 0.20670083978720682 0 rpy=1 0 0
- joint j0_j1: origin xyz=0 -0.27224610714888436 0 rpy=1 0 0 -> xyz=0 -0.23362430842753437 0 rpy=1 0 0
- joint k0_k1: origin xyz=0 0 0.5321029169218512 rpy=1 0 0 -> xyz=0 0 0.8581481960782829 rpy=1 0 0

File: body1.urdf (robot description, URDF)
Before this commit: robot robot, 7 links, 6 joints
Links:
- link Torso: geometry collision box size=0.4270820660990066 1.0538899660439736 1.152347599706828; visual box size=0.4270820660990066 1.0538899660439736 1.152347599706828
- link i0: geometry collision box size=0.4662786948372766 0.20670083978720682 0.24069037165999171; visual box size=0.4662786948372766 0.20670083978720682 0.24069037165999171
- link i1: geometry collision box size=0.42713318362025565 0.9490551511654679 0.6150144779125608; visual box size=0.42713318362025565 0.9490551511654679 0.6150144779125608
- link j0: geometry collision box size=0.3508349298730473 0.23362430842753437 0.8934338651499589; visual box size=0.3508349298730473 0.23362430842753437 0.8934338651499589
- link j1: geometry collision box size=0.847778629833061 0.6659606540101592 0.9166403317259235; visual box size=0.847778629833061 0.6659606540101592 0.9166403317259235
- link k0: geometry collision box size=0.6140921707159852 0.6159897364099624 0.8581481960782829; visual box size=0.6140921707159852 0.6159897364099624 0.8581481960782829
- link k1: geometry collision box size=0.8083844113766532 0.7965283546037021 0.814354034299329; visual box size=0.8083844113766532 0.7965283546037021 0.814354034299329
Joints:
- joint Torso_i0: origin xyz=0 0.6195807324398217 1.5279984833440365 rpy=0 0 0 -> xyz=0 0.5269449830219868 1.728521399560242 rpy=0 0 0
- joint Torso_j0: origin xyz=0 -0.6195807324398217 1.5279984833440365 rpy=0 0 1 -> xyz=0 -0.5269449830219868 1.728521399560242 rpy=0 0 1
- joint Torso_k0: origin xyz=0 0 2.037331311125382 rpy=0 0 1 -> xyz=0 0 2.304695199413656 rpy=0 0 1
- joint i0_i1: origin xyz=0 0.9898086850351462 0 rpy=1 0 0 -> xyz=0 0.20670083978720682 0 rpy=1 0 0
- joint j0_j1: origin xyz=0 -0.27224610714888436 0 rpy=1 0 0 -> xyz=0 -0.23362430842753437 0 rpy=1 0 0
- joint k0_k1: origin xyz=0 0 0.5321029169218512 rpy=1 0 0 -> xyz=0 0 0.8581481960782829 rpy=1 0 0

File: body3.urdf (robot description, URDF)
Before this commit: robot robot, 7 links, 6 joints
Links:
- link Torso: geometry collision box size=0.4270820660990066 1.0538899660439736 1.152347599706828; visual box size=0.4270820660990066 1.0538899660439736 1.152347599706828
- link i0: geometry collision box size=0.4662786948372766 0.20670083978720682 0.24069037165999171; visual box size=0.4662786948372766 0.20670083978720682 0.24069037165999171
- link i1: geometry collision box size=0.42713318362025565 0.9490551511654679 0.6150144779125608; visual box size=0.42713318362025565 0.9490551511654679 0.6150144779125608
- link j0: geometry collision box size=0.3508349298730473 0.23362430842753437 0.8934338651499589; visual box size=0.3508349298730473 0.23362430842753437 0.8934338651499589
- link j1: geometry collision box size=0.847778629833061 0.6659606540101592 0.9166403317259235; visual box size=0.847778629833061 0.6659606540101592 0.9166403317259235
- link k0: geometry collision box size=0.6140921707159852 0.6159897364099624 0.8581481960782829; visual box size=0.6140921707159852 0.6159897364099624 0.8581481960782829
- link k1: geometry collision box size=0.8083844113766532 0.7965283546037021 0.814354034299329; visual box size=0.8083844113766532 0.7965283546037021 0.814354034299329
Joints:
- joint Torso_i0: origin xyz=0 0.6195807324398217 1.5279984833440365 rpy=0 0 0 -> xyz=0 0.5269449830219868 1.728521399560242 rpy=1 0 0
- joint Torso_j0: origin xyz=0 -0.6195807324398217 1.5279984833440365 rpy=0 0 1 -> xyz=0 -0.5269449830219868 1.728521399560242 rpy=0 0 1
- joint Torso_k0: origin xyz=0 0 2.037331311125382 rpy=0 0 1 -> xyz=0 0 2.304695199413656 rpy=0 0 1
- joint i0_i1: origin xyz=0 0.9898086850351462 0 rpy=1 0 0 -> xyz=0 0.20670083978720682 0 rpy=1 0 0
- joint j0_j1: origin xyz=0 -0.27224610714888436 0 rpy=1 0 0 -> xyz=0 -0.23362430842753437 0 rpy=1 0 0
- joint k0_k1: origin xyz=0 0 0.5321029169218512 rpy=1 0 0 -> xyz=0 0 0.8581481960782829 rpy=1 0 0

File: body4.urdf (robot description, URDF)
Before this commit: robot robot, 7 links, 6 joints
Links:
- link Torso: geometry collision box size=0.4270820660990066 1.0538899660439736 1.152347599706828; visual box size=0.4270820660990066 1.0538899660439736 1.152347599706828
- link i0: geometry collision box size=0.4662786948372766 0.20670083978720682 0.24069037165999171; visual box size=0.4662786948372766 0.20670083978720682 0.24069037165999171
- link i1: geometry collision box size=0.42713318362025565 0.9490551511654679 0.6150144779125608; visual box size=0.42713318362025565 0.9490551511654679 0.6150144779125608
- link j0: geometry collision box size=0.3508349298730473 0.23362430842753437 0.8934338651499589; visual box size=0.3508349298730473 0.23362430842753437 0.8934338651499589
- link j1: geometry collision box size=0.847778629833061 0.6659606540101592 0.9166403317259235; visual box size=0.847778629833061 0.6659606540101592 0.9166403317259235
- link k0: geometry collision box size=0.6140921707159852 0.6159897364099624 0.8581481960782829; visual box size=0.6140921707159852 0.6159897364099624 0.8581481960782829
- link k1: geometry collision box size=0.8083844113766532 0.7965283546037021 0.814354034299329; visual box size=0.8083844113766532 0.7965283546037021 0.814354034299329
Joints:
- joint Torso_i0: origin xyz=0 0.6195807324398217 1.5279984833440365 rpy=0 0 1 -> xyz=0 0.5269449830219868 1.728521399560242 rpy=0 0 1
- joint Torso_j0: origin xyz=0 -0.6195807324398217 1.5279984833440365 rpy=0 0 1 -> xyz=0 -0.5269449830219868 1.728521399560242 rpy=0 0 1
- joint Torso_k0: origin xyz=0 0 2.037331311125382 rpy=0 0 1 -> xyz=0 0 2.304695199413656 rpy=0 0 1
- joint i0_i1: origin xyz=0 0.9898086850351462 0 rpy=1 0 0 -> xyz=0 0.20670083978720682 0 rpy=1 0 0
- joint j0_j1: origin xyz=0 -0.27224610714888436 0 rpy=1 0 0 -> xyz=0 -0.23362430842753437 0 rpy=1 0 0
- joint k0_k1: origin xyz=0 0 0.5321029169218512 rpy=1 0 0 -> xyz=0 0 0.8581481960782829 rpy=1 0 0

File: body5.urdf (robot description, URDF)
Before this commit: robot robot, 7 links, 6 joints
Links:
- link Torso: geometry collision box size=0.4270820660990066 1.0538899660439736 1.152347599706828; visual box size=0.4270820660990066 1.0538899660439736 1.152347599706828
- link i0: geometry collision box size=0.4662786948372766 0.20670083978720682 0.24069037165999171; visual box size=0.4662786948372766 0.20670083978720682 0.24069037165999171
- link i1: geometry collision box size=0.42713318362025565 0.9490551511654679 0.6150144779125608; visual box size=0.42713318362025565 0.9490551511654679 0.6150144779125608
- link j0: geometry collision box size=0.3508349298730473 0.23362430842753437 0.8934338651499589; visual box size=0.3508349298730473 0.23362430842753437 0.8934338651499589
- link j1: geometry collision box size=0.847778629833061 0.6659606540101592 0.9166403317259235; visual box size=0.847778629833061 0.6659606540101592 0.9166403317259235
- link k0: geometry collision box size=0.6140921707159852 0.6159897364099624 0.8581481960782829; visual box size=0.6140921707159852 0.6159897364099624 0.8581481960782829
- link k1: geometry collision box size=0.8083844113766532 0.7965283546037021 0.814354034299329; visual box size=0.8083844113766532 0.7965283546037021 0.814354034299329
Joints:
- joint Torso_i0: origin xyz=0 0.6195807324398217 1.5279984833440365 rpy=1 0 0 -> xyz=0 0.5269449830219868 1.728521399560242 rpy=1 0 0
- joint Torso_j0: origin xyz=0 -0.6195807324398217 1.5279984833440365 rpy=0 0 1 -> xyz=0 -0.5269449830219868 1.728521399560242 rpy=0 0 1
- joint Torso_k0: origin xyz=0 0 2.037331311125382 rpy=0 0 1 -> xyz=0 0 2.304695199413656 rpy=0 0 1
- joint i0_i1: origin xyz=0 0.9898086850351462 0 rpy=1 0 0 -> xyz=0 0.20670083978720682 0 rpy=1 0 0
- joint j0_j1: origin xyz=0 -0.27224610714888436 0 rpy=1 0 0 -> xyz=0 -0.23362430842753437 0 rpy=1 0 0
- joint k0_k1: origin xyz=0 0 0.5321029169218512 rpy=1 0 0 -> xyz=0 0 0.8581481960782829 rpy=1 0 0

Commit message: add,remove,change size now working

File: body0.urdf (robot description, URDF)
Before this commit: robot robot, 7 links, 6 joints
Links:
- link Torso: geometry collision box size=0.5356045539707158 1.1904291023214877 1.071429813023242; visual box size=0.5356045539707158 1.1904291023214877 1.071429813023242
- link i0: geometry collision box size=0.40924316883828066 0.6589015736985113 0.26448349968284124; visual box size=0.40924316883828066 0.6589015736985113 0.26448349968284124
- link i1: geometry collision box size=0.8058847319685489 0.6800640711286877 0.8595753567746054; visual box size=0.8058847319685489 0.6800640711286877 0.8595753567746054
- link j0: geometry collision box size=0.5689011552906347 0.33601907743104975 0.5903568235372258; visual box size=0.5689011552906347 0.33601907743104975 0.5903568235372258
- link j1: geometry collision box size=0.48108765788658436 0.9478584436329305 0.9335598339230726; visual box size=0.48108765788658436 0.9478584436329305 0.9335598339230726
- link k0: geometry collision box size=0.710791078586887 0.9884323070003995 0.992919956546358; visual box size=0.710791078586887 0.9884323070003995 0.992919956546358
- link k1: geometry collision box size=0.29962249028094706 0.7401689396409865 0.4893130437560174; visual box size=0.29962249028094706 0.7401689396409865 0.4893130437560174
Joints:
- joint Torso_i0: origin xyz=0 0.5269449830219868 1.728521399560242 rpy=1 0 0 -> xyz=0 0.5952145511607438 1.6071447195348632 rpy=0 1 0
- joint Torso_j0: origin xyz=0 -0.5269449830219868 1.728521399560242 rpy=0 0 1 -> xyz=0 -0.5952145511607438 1.6071447195348632 rpy=0 0 1
- joint Torso_k0: origin xyz=0 0 2.304695199413656 rpy=0 0 1 -> xyz=0 0 2.142859626046484 rpy=0 0 1
- joint i0_i1: origin xyz=0 0.20670083978720682 0 rpy=1 0 0 -> xyz=0 0.6589015736985113 0 rpy=1 0 0
- joint j0_j1: origin xyz=0 -0.23362430842753437 0 rpy=1 0 0 -> xyz=0 -0.33601907743104975 0 rpy=1 0 0
- joint k0_k1: origin xyz=0 0 0.8581481960782829 rpy=1 0 0 -> xyz=0 0 0.992919956546358 rpy=1 0 0

File: body1.urdf (robot description, URDF)
Before this commit: robot robot, 7 links, 6 joints
Links:
- link Torso: geometry collision box size=0.5356045539707158 1.1904291023214877 1.071429813023242; visual box size=0.5356045539707158 1.1904291023214877 1.071429813023242
- link i0: geometry collision box size=0.40924316883828066 0.6589015736985113 0.26448349968284124; visual box size=0.40924316883828066 0.6589015736985113 0.26448349968284124
- link i1: geometry collision box size=0.8058847319685489 0.6800640711286877 0.8595753567746054; visual box size=0.8058847319685489 0.6800640711286877 0.8595753567746054
- link j0: geometry collision box size=0.5689011552906347 0.33601907743104975 0.5903568235372258; visual box size=0.5689011552906347 0.33601907743104975 0.5903568235372258
- link j1: geometry collision box size=0.48108765788658436 0.9478584436329305 0.9335598339230726; visual box size=0.48108765788658436 0.9478584436329305 0.9335598339230726
- link k0: geometry collision box size=0.710791078586887 0.9884323070003995 0.992919956546358; visual box size=0.710791078586887 0.9884323070003995 0.992919956546358
- link k1: geometry collision box size=0.29962249028094706 0.7401689396409865 0.4893130437560174; visual box size=0.29962249028094706 0.7401689396409865 0.4893130437560174
Joints:
- joint Torso_i0: origin xyz=0 0.5269449830219868 1.728521399560242 rpy=0 0 0 -> xyz=0 0.5952145511607438 1.6071447195348632 rpy=0 0 0
- joint Torso_j0: origin xyz=0 -0.5269449830219868 1.728521399560242 rpy=0 0 1 -> xyz=0 -0.5952145511607438 1.6071447195348632 rpy=0 0 1
- joint Torso_k0: origin xyz=0 0 2.304695199413656 rpy=0 0 1 -> xyz=0 0 2.142859626046484 rpy=0 0 1
- joint i0_i1: origin xyz=0 0.20670083978720682 0 rpy=1 0 0 -> xyz=0 0.6589015736985113 0 rpy=1 0 0
- joint j0_j1: origin xyz=0 -0.23362430842753437 0 rpy=1 0 0 -> xyz=0 -0.33601907743104975 0 rpy=1 0 0
- joint k0_k1: origin xyz=0 0 0.8581481960782829 rpy=1 0 0 -> xyz=0 0 0.992919956546358 rpy=1 0 0

File: body2.urdf (robot description, URDF)
Before this commit: robot robot, 7 links, 6 joints
Links:
- link Torso: geometry collision box size=0.5356045539707158 1.1904291023214877 1.071429813023242; visual box size=0.5356045539707158 1.1904291023214877 1.071429813023242
- link i0: geometry collision box size=0.40924316883828066 0.6589015736985113 0.26448349968284124; visual box size=0.40924316883828066 0.6589015736985113 0.26448349968284124
- link i1: geometry collision box size=0.8058847319685489 0.6800640711286877 0.8595753567746054; visual box size=0.8058847319685489 0.6800640711286877 0.8595753567746054
- link j0: geometry collision box size=0.5689011552906347 0.33601907743104975 0.5903568235372258; visual box size=0.5689011552906347 0.33601907743104975 0.5903568235372258
- link j1: geometry collision box size=0.48108765788658436 0.9478584436329305 0.9335598339230726; visual box size=0.48108765788658436 0.9478584436329305 0.9335598339230726
- link k0: geometry collision box size=0.710791078586887 0.9884323070003995 0.992919956546358; visual box size=0.710791078586887 0.9884323070003995 0.992919956546358
- link k1: geometry collision box size=0.29962249028094706 0.7401689396409865 0.4893130437560174; visual box size=0.29962249028094706 0.7401689396409865 0.4893130437560174
Joints:
- joint Torso_i0: origin xyz=0 0.5269449830219868 1.728521399560242 rpy=1 0 0 -> xyz=0 0.5952145511607438 1.6071447195348632 rpy=0 0 0
- joint Torso_j0: origin xyz=0 -0.5269449830219868 1.728521399560242 rpy=0 0 1 -> xyz=0 -0.5952145511607438 1.6071447195348632 rpy=0 0 1
- joint Torso_k0: origin xyz=0 0 2.304695199413656 rpy=0 0 1 -> xyz=0 0 2.142859626046484 rpy=0 0 1
- joint i0_i1: origin xyz=0 0.20670083978720682 0 rpy=1 0 0 -> xyz=0 0.6589015736985113 0 rpy=1 0 0
- joint j0_j1: origin xyz=0 -0.23362430842753437 0 rpy=1 0 0 -> xyz=0 -0.33601907743104975 0 rpy=1 0 0
- joint k0_k1: origin xyz=0 0 0.8581481960782829 rpy=1 0 0 -> xyz=0 0 0.992919956546358 rpy=1 0 0

File: body4.urdf (robot description, URDF)
Before this commit: robot robot, 7 links, 6 joints
Links:
- link Torso: geometry collision box size=0.5356045539707158 1.1904291023214877 1.071429813023242; visual box size=0.5356045539707158 1.1904291023214877 1.071429813023242
- link i0: geometry collision box size=0.40924316883828066 0.6589015736985113 0.26448349968284124; visual box size=0.40924316883828066 0.6589015736985113 0.26448349968284124
- link i1: geometry collision box size=0.8058847319685489 0.6800640711286877 0.8595753567746054; visual box size=0.8058847319685489 0.6800640711286877 0.8595753567746054
- link j0: geometry collision box size=0.5689011552906347 0.33601907743104975 0.5903568235372258; visual box size=0.5689011552906347 0.33601907743104975 0.5903568235372258
- link j1: geometry collision box size=0.48108765788658436 0.9478584436329305 0.9335598339230726; visual box size=0.48108765788658436 0.9478584436329305 0.9335598339230726
- link k0: geometry collision box size=0.710791078586887 0.9884323070003995 0.992919956546358; visual box size=0.710791078586887 0.9884323070003995 0.992919956546358
- link k1: geometry collision box size=0.29962249028094706 0.7401689396409865 0.4893130437560174; visual box size=0.29962249028094706 0.7401689396409865 0.4893130437560174
Joints:
- joint Torso_i0: origin xyz=0 0.5269449830219868 1.728521399560242 rpy=0 0 1 -> xyz=0 0.5952145511607438 1.6071447195348632 rpy=1 0 0
- joint Torso_j0: origin xyz=0 -0.5269449830219868 1.728521399560242 rpy=0 0 1 -> xyz=0 -0.5952145511607438 1.6071447195348632 rpy=0 0 1
- joint Torso_k0: origin xyz=0 0 2.304695199413656 rpy=0 0 1 -> xyz=0 0 2.142859626046484 rpy=0 0 1
- joint i0_i1: origin xyz=0 0.20670083978720682 0 rpy=1 0 0 -> xyz=0 0.6589015736985113 0 rpy=1 0 0
- joint j0_j1: origin xyz=0 -0.23362430842753437 0 rpy=1 0 0 -> xyz=0 -0.33601907743104975 0 rpy=1 0 0
- joint k0_k1: origin xyz=0 0 0.8581481960782829 rpy=1 0 0 -> xyz=0 0 0.992919956546358 rpy=1 0 0

File: body5.urdf (robot description, URDF)
Before this commit: robot robot, 7 links, 6 joints
Links:
- removed link j1
- removed link k1
- link Torso: geometry collision box size=0.5356045539707158 1.1904291023214877 1.071429813023242; visual box size=0.5356045539707158 1.1904291023214877 1.071429813023242
- link i0: geometry collision box size=0.40924316883828066 0.6589015736985113 0.26448349968284124; visual box size=0.40924316883828066 0.6589015736985113 0.26448349968284124
- link i1: geometry collision box size=0.8058847319685489 0.6800640711286877 0.8595753567746054; visual box size=0.8058847319685489 0.6800640711286877 0.8595753567746054
- link j0: geometry collision box size=0.5689011552906347 0.33601907743104975 0.5903568235372258; visual box size=0.5689011552906347 0.33601907743104975 0.5903568235372258
- link k0: geometry collision box size=0.710791078586887 0.9884323070003995 0.992919956546358; visual box size=0.710791078586887 0.9884323070003995 0.992919956546358
Joints:
- removed joint j0_j1
- removed joint k0_k1
- joint Torso_i0: origin xyz=0 0.5269449830219868 1.728521399560242 rpy=1 0 0 -> xyz=0 0.5952145511607438 1.6071447195348632 rpy=0 0 0
- joint Torso_j0: origin xyz=0 -0.5269449830219868 1.728521399560242 rpy=0 0 1 -> xyz=0 -0.5952145511607438 1.6071447195348632 rpy=0 0 1
- joint Torso_k0: origin xyz=0 0 2.304695199413656 rpy=0 0 1 -> xyz=0 0 2.142859626046484 rpy=0 0 1
- joint i0_i1: origin xyz=0 0.20670083978720682 0 rpy=1 0 0 -> xyz=0 0.6589015736985113 0 rpy=1 0 0
