Commit message: why arent my joints working >:(

File: body0.urdf (robot description, URDF)
Before this commit: robot robot, 7 links, 6 joints
Links:
- link Torso: geometry collision box size=0.7270228655515488 0.7292258214042837 1.1258217221794715; visual box size=0.7270228655515488 0.7292258214042837 1.1258217221794715
- link i0: geometry collision box size=0.2244946194776435 0.8671980434301998 0.44899747028739334; visual box size=0.2244946194776435 0.8671980434301998 0.44899747028739334
- link i1: geometry collision box size=0.8310824608995113 0.24893751158378974 0.6868873738781187; visual box size=0.8310824608995113 0.24893751158378974 0.6868873738781187
- link j0: geometry collision box size=0.5756628666602228 0.7392876657518792 0.31631609887733225; visual box size=0.5756628666602228 0.7392876657518792 0.31631609887733225
- link j1: geometry collision box size=0.995159994125997 0.6275858017941741 0.6060072164258576; visual box size=0.995159994125997 0.6275858017941741 0.6060072164258576
- link k0: geometry collision box size=0.3603192808325041 0.8881112222223901 0.4752483356864448; visual box size=0.3603192808325041 0.8881112222223901 0.4752483356864448
- link k1: geometry collision box size=0.8203947820122648 0.4270699520020683 0.3215233129628592; visual box size=0.8203947820122648 0.4270699520020683 0.3215233129628592
Joints:
- joint Torso_i0: origin xyz=0 0.5952145511607438 1.6071447195348632 rpy=0 1 0 -> xyz=0 0.36461291070214186 1.6887325832692073 rpy=1 0 0
- joint Torso_j0: origin xyz=0 -0.5952145511607438 1.6071447195348632 rpy=0 0 1 -> xyz=0 -0.36461291070214186 1.6887325832692073 rpy=0 0 1
- joint Torso_k0: origin xyz=0 0 2.142859626046484 rpy=0 0 1 -> xyz=0 0 2.251643444358943 rpy=0 0 1
- joint i0_i1: origin xyz=0 0.6589015736985113 0 rpy=1 0 0 -> xyz=0 0.8671980434301998 0 rpy=1 0 0
- joint j0_j1: origin xyz=0 -0.33601907743104975 0 rpy=1 0 0 -> xyz=0 -0.7392876657518792 0 rpy=1 0 0
- joint k0_k1: origin xyz=0 0 0.992919956546358 rpy=1 0 0 -> xyz=0 0 0.4752483356864448 rpy=1 0 0

File: body1.urdf (robot description, URDF)
Before this commit: robot robot, 7 links, 6 joints
Links:
- link Torso: geometry collision box size=0.7270228655515488 0.7292258214042837 1.1258217221794715; visual box size=0.7270228655515488 0.7292258214042837 1.1258217221794715
- link i0: geometry collision box size=0.2244946194776435 0.8671980434301998 0.44899747028739334; visual box size=0.2244946194776435 0.8671980434301998 0.44899747028739334
- link i1: geometry collision box size=0.8310824608995113 0.24893751158378974 0.6868873738781187; visual box size=0.8310824608995113 0.24893751158378974 0.6868873738781187
- link j0: geometry collision box size=0.5756628666602228 0.7392876657518792 0.31631609887733225; visual box size=0.5756628666602228 0.7392876657518792 0.31631609887733225
- link j1: geometry collision box size=0.995159994125997 0.6275858017941741 0.6060072164258576; visual box size=0.995159994125997 0.6275858017941741 0.6060072164258576
- link k0: geometry collision box size=0.3603192808325041 0.8881112222223901 0.4752483356864448; visual box size=0.3603192808325041 0.8881112222223901 0.4752483356864448
- link k1: geometry collision box size=0.8203947820122648 0.4270699520020683 0.3215233129628592; visual box size=0.8203947820122648 0.4270699520020683 0.3215233129628592
Joints:
- joint Torso_i0: origin xyz=0 0.5952145511607438 1.6071447195348632 rpy=0 0 0 -> xyz=0 0.36461291070214186 1.6887325832692073 rpy=0 0 1
- joint Torso_j0: origin xyz=0 -0.5952145511607438 1.6071447195348632 rpy=0 0 1 -> xyz=0 -0.36461291070214186 1.6887325832692073 rpy=0 0 1
- joint Torso_k0: origin xyz=0 0 2.142859626046484 rpy=0 0 1 -> xyz=0 0 2.251643444358943 rpy=0 0 1
- joint i0_i1: origin xyz=0 0.6589015736985113 0 rpy=1 0 0 -> xyz=0 0.8671980434301998 0 rpy=1 0 0
- joint j0_j1: origin xyz=0 -0.33601907743104975 0 rpy=1 0 0 -> xyz=0 -0.7392876657518792 0 rpy=1 0 0
- joint k0_k1: origin xyz=0 0 0.992919956546358 rpy=1 0 0 -> xyz=0 0 0.4752483356864448 rpy=1 0 0

File: body2.urdf (robot description, URDF)
Before this commit: robot robot, 7 links, 6 joints
Links:
- link Torso: geometry collision box size=0.7270228655515488 0.7292258214042837 1.1258217221794715; visual box size=0.7270228655515488 0.7292258214042837 1.1258217221794715
- link i0: geometry collision box size=0.2244946194776435 0.8671980434301998 0.44899747028739334; visual box size=0.2244946194776435 0.8671980434301998 0.44899747028739334
- link i1: geometry collision box size=0.8310824608995113 0.24893751158378974 0.6868873738781187; visual box size=0.8310824608995113 0.24893751158378974 0.6868873738781187
- link j0: geometry collision box size=0.5756628666602228 0.7392876657518792 0.31631609887733225; visual box size=0.5756628666602228 0.7392876657518792 0.31631609887733225
- link j1: geometry collision box size=0.995159994125997 0.6275858017941741 0.6060072164258576; visual box size=0.995159994125997 0.6275858017941741 0.6060072164258576
- link k0: geometry collision box size=0.3603192808325041 0.8881112222223901 0.4752483356864448; visual box size=0.3603192808325041 0.8881112222223901 0.4752483356864448
- link k1: geometry collision box size=0.8203947820122648 0.4270699520020683 0.3215233129628592; visual box size=0.8203947820122648 0.4270699520020683 0.3215233129628592
Joints:
- joint Torso_i0: origin xyz=0 0.5952145511607438 1.6071447195348632 rpy=0 0 0 -> xyz=0 0.36461291070214186 1.6887325832692073 rpy=0 1 0
- joint Torso_j0: origin xyz=0 -0.5952145511607438 1.6071447195348632 rpy=0 0 1 -> xyz=0 -0.36461291070214186 1.6887325832692073 rpy=0 0 1
- joint Torso_k0: origin xyz=0 0 2.142859626046484 rpy=0 0 1 -> xyz=0 0 2.251643444358943 rpy=0 0 1
- joint i0_i1: origin xyz=0 0.6589015736985113 0 rpy=1 0 0 -> xyz=0 0.8671980434301998 0 rpy=1 0 0
- joint j0_j1: origin xyz=0 -0.33601907743104975 0 rpy=1 0 0 -> xyz=0 -0.7392876657518792 0 rpy=1 0 0
- joint k0_k1: origin xyz=0 0 0.992919956546358 rpy=1 0 0 -> xyz=0 0 0.4752483356864448 rpy=1 0 0

File: body3.urdf (robot description, URDF)
Before this commit: robot robot, 7 links, 6 joints
Links:
- link Torso: geometry collision box size=0.7270228655515488 0.7292258214042837 1.1258217221794715; visual box size=0.7270228655515488 0.7292258214042837 1.1258217221794715
- link i0: geometry collision box size=0.2244946194776435 0.8671980434301998 0.44899747028739334; visual box size=0.2244946194776435 0.8671980434301998 0.44899747028739334
- link i1: geometry collision box size=0.8310824608995113 0.24893751158378974 0.6868873738781187; visual box size=0.8310824608995113 0.24893751158378974 0.6868873738781187
- link j0: geometry collision box size=0.5756628666602228 0.7392876657518792 0.31631609887733225; visual box size=0.5756628666602228 0.7392876657518792 0.31631609887733225
- link j1: geometry collision box size=0.995159994125997 0.6275858017941741 0.6060072164258576; visual box size=0.995159994125997 0.6275858017941741 0.6060072164258576
- link k0: geometry collision box size=0.3603192808325041 0.8881112222223901 0.4752483356864448; visual box size=0.3603192808325041 0.8881112222223901 0.4752483356864448
- link k1: geometry collision box size=0.8203947820122648 0.4270699520020683 0.3215233129628592; visual box size=0.8203947820122648 0.4270699520020683 0.3215233129628592
Joints:
- joint Torso_i0: origin xyz=0 0.5952145511607438 1.6071447195348632 rpy=0 0 0 -> xyz=0 0.36461291070214186 1.6887325832692073 rpy=1 0 0
- joint Torso_j0: origin xyz=0 -0.5952145511607438 1.6071447195348632 rpy=0 0 1 -> xyz=0 -0.36461291070214186 1.6887325832692073 rpy=0 0 1
- joint Torso_k0: origin xyz=0 0 2.142859626046484 rpy=0 0 1 -> xyz=0 0 2.251643444358943 rpy=0 0 1
- joint i0_i1: origin xyz=0 0.6589015736985113 0 rpy=1 0 0 -> xyz=0 0.8671980434301998 0 rpy=1 0 0
- joint j0_j1: origin xyz=0 -0.33601907743104975 0 rpy=1 0 0 -> xyz=0 -0.7392876657518792 0 rpy=1 0 0
- joint k0_k1: origin xyz=0 0 0.992919956546358 rpy=1 0 0 -> xyz=0 0 0.4752483356864448 rpy=1 0 0

File: body4.urdf (robot description, URDF)
Before this commit: robot robot, 7 links, 6 joints
Links:
- link Torso: geometry collision box size=0.7270228655515488 0.7292258214042837 1.1258217221794715; visual box size=0.7270228655515488 0.7292258214042837 1.1258217221794715
- link i0: geometry collision box size=0.2244946194776435 0.8671980434301998 0.44899747028739334; visual box size=0.2244946194776435 0.8671980434301998 0.44899747028739334
- link i1: geometry collision box size=0.8310824608995113 0.24893751158378974 0.6868873738781187; visual box size=0.8310824608995113 0.24893751158378974 0.6868873738781187
- link j0: geometry collision box size=0.5756628666602228 0.7392876657518792 0.31631609887733225; visual box size=0.5756628666602228 0.7392876657518792 0.31631609887733225
- link j1: geometry collision box size=0.995159994125997 0.6275858017941741 0.6060072164258576; visual box size=0.995159994125997 0.6275858017941741 0.6060072164258576
- link k0: geometry collision box size=0.3603192808325041 0.8881112222223901 0.4752483356864448; visual box size=0.3603192808325041 0.8881112222223901 0.4752483356864448
- link k1: geometry collision box size=0.8203947820122648 0.4270699520020683 0.3215233129628592; visual box size=0.8203947820122648 0.4270699520020683 0.3215233129628592
Joints:
- joint Torso_i0: origin xyz=0 0.5952145511607438 1.6071447195348632 rpy=1 0 0 -> xyz=0 0.36461291070214186 1.6887325832692073 rpy=0 0 0
- joint Torso_j0: origin xyz=0 -0.5952145511607438 1.6071447195348632 rpy=0 0 1 -> xyz=0 -0.36461291070214186 1.6887325832692073 rpy=0 0 1
- joint Torso_k0: origin xyz=0 0 2.142859626046484 rpy=0 0 1 -> xyz=0 0 2.251643444358943 rpy=0 0 1
- joint i0_i1: origin xyz=0 0.6589015736985113 0 rpy=1 0 0 -> xyz=0 0.8671980434301998 0 rpy=1 0 0
- joint j0_j1: origin xyz=0 -0.33601907743104975 0 rpy=1 0 0 -> xyz=0 -0.7392876657518792 0 rpy=1 0 0
- joint k0_k1: origin xyz=0 0 0.992919956546358 rpy=1 0 0 -> xyz=0 0 0.4752483356864448 rpy=1 0 0

File: body5.urdf (robot description, URDF)
Before this commit: robot robot, 5 links, 4 joints
Links:
- added link j1, mass 1; collision box size=0.995159994125997 0.6275858017941741 0.6060072164258576; visual box size=0.995159994125997 0.6275858017941741 0.6060072164258576
- added link k1, mass 1; collision box size=0.8203947820122648 0.4270699520020683 0.3215233129628592; visual box size=0.8203947820122648 0.4270699520020683 0.3215233129628592
- link Torso: geometry collision box size=0.7270228655515488 0.7292258214042837 1.1258217221794715; visual box size=0.7270228655515488 0.7292258214042837 1.1258217221794715
- link i0: geometry collision box size=0.2244946194776435 0.8671980434301998 0.44899747028739334; visual box size=0.2244946194776435 0.8671980434301998 0.44899747028739334
- link i1: geometry collision box size=0.8310824608995113 0.24893751158378974 0.6868873738781187; visual box size=0.8310824608995113 0.24893751158378974 0.6868873738781187
- link j0: geometry collision box size=0.5756628666602228 0.7392876657518792 0.31631609887733225; visual box size=0.5756628666602228 0.7392876657518792 0.31631609887733225
- link k0: geometry collision box size=0.3603192808325041 0.8881112222223901 0.4752483356864448; visual box size=0.3603192808325041 0.8881112222223901 0.4752483356864448
Joints:
- added joint j0_j1: type revolute, parent j0, child j1, origin xyz=0 -0.7392876657518792 0 rpy=1 0 0, axis 1 0 0, limit lower=-3.14159 upper=3.14159 effort=0.0 velocity=0.0
- added joint k0_k1: type revolute, parent k0, child k1, origin xyz=0 0 0.4752483356864448 rpy=1 0 0, axis 1 0 0, limit lower=-3.14159 upper=3.14159 effort=0.0 velocity=0.0
- joint Torso_i0: origin xyz=0 0.5952145511607438 1.6071447195348632 rpy=0 0 0 -> xyz=0 0.36461291070214186 1.6887325832692073 rpy=0 1 0
- joint Torso_j0: origin xyz=0 -0.5952145511607438 1.6071447195348632 rpy=0 0 1 -> xyz=0 -0.36461291070214186 1.6887325832692073 rpy=0 0 1
- joint Torso_k0: origin xyz=0 0 2.142859626046484 rpy=0 0 1 -> xyz=0 0 2.251643444358943 rpy=0 0 1
- joint i0_i1: origin xyz=0 0.6589015736985113 0 rpy=1 0 0 -> xyz=0 0.8671980434301998 0 rpy=1 0 0

File: body6.urdf (robot description, URDF)
Before this commit: robot robot, 8 links, 7 joints
Links:
- removed link i2
- removed link j2
- added link k1, mass 1; collision box size=0.8203947820122648 0.4270699520020683 0.3215233129628592; visual box size=0.8203947820122648 0.4270699520020683 0.3215233129628592
- link Torso: geometry collision box size=0.7270228655515488 0.7292258214042837 1.1258217221794715; visual box size=0.7270228655515488 0.7292258214042837 1.1258217221794715
- link i0: geometry collision box size=0.2244946194776435 0.8671980434301998 0.44899747028739334; visual box size=0.2244946194776435 0.8671980434301998 0.44899747028739334
- link i1: geometry collision box size=0.8310824608995113 0.24893751158378974 0.6868873738781187; visual box size=0.8310824608995113 0.24893751158378974 0.6868873738781187
- link j0: geometry collision box size=0.5756628666602228 0.7392876657518792 0.31631609887733225; visual box size=0.5756628666602228 0.7392876657518792 0.31631609887733225
- link j1: geometry collision box size=0.995159994125997 0.6275858017941741 0.6060072164258576; visual box size=0.995159994125997 0.6275858017941741 0.6060072164258576
- link k0: geometry collision box size=0.3603192808325041 0.8881112222223901 0.4752483356864448; visual box size=0.3603192808325041 0.8881112222223901 0.4752483356864448
Joints:
- removed joint i1_i2
- removed joint j1_j2
- added joint k0_k1: type revolute, parent k0, child k1, origin xyz=0 0 0.4752483356864448 rpy=1 0 0, axis 1 0 0, limit lower=-3.14159 upper=3.14159 effort=0.0 velocity=0.0
- joint Torso_i0: origin xyz=0 0.3751240526539688 0.6968726327450769 rpy=1 0 0 -> xyz=0 0.36461291070214186 1.6887325832692073 rpy=0 1 0
- joint Torso_j0: origin xyz=0 -0.3751240526539688 0.6968726327450769 rpy=0 0 1 -> xyz=0 -0.36461291070214186 1.6887325832692073 rpy=0 0 1
- joint Torso_k0: origin xyz=0 0 0.9291635103267692 rpy=0 0 1 -> xyz=0 0 2.251643444358943 rpy=0 0 1
- joint i0_i1: origin xyz=0 0.6362546528634063 0 rpy=1 0 0 -> xyz=0 0.8671980434301998 0 rpy=1 0 0
- joint j0_j1: origin xyz=0 -0.5195416040203034 0 rpy=1 0 0 -> xyz=0 -0.7392876657518792 0 rpy=1 0 0

File: body8.urdf (robot description, URDF)
Before this commit: robot robot, 2 links, 1 joints
Links:
- added link i1, mass 1; collision box size=0.8310824608995113 0.24893751158378974 0.6868873738781187; visual box size=0.8310824608995113 0.24893751158378974 0.6868873738781187
- added link j0, mass 1; collision box size=0.5756628666602228 0.7392876657518792 0.31631609887733225; visual box size=0.5756628666602228 0.7392876657518792 0.31631609887733225
- added link j1, mass 1; collision box size=0.995159994125997 0.6275858017941741 0.6060072164258576; visual box size=0.995159994125997 0.6275858017941741 0.6060072164258576
- added link k0, mass 1; collision box size=0.3603192808325041 0.8881112222223901 0.4752483356864448; visual box size=0.3603192808325041 0.8881112222223901 0.4752483356864448
- added link k1, mass 1; collision box size=0.8203947820122648 0.4270699520020683 0.3215233129628592; visual box size=0.8203947820122648 0.4270699520020683 0.3215233129628592
- link Torso: geometry collision box size=0.7270228655515488 0.7292258214042837 1.1258217221794715; visual box size=0.7270228655515488 0.7292258214042837 1.1258217221794715
- link i0: geometry collision box size=0.2244946194776435 0.8671980434301998 0.44899747028739334; visual box size=0.2244946194776435 0.8671980434301998 0.44899747028739334
Joints:
- added joint Torso_j0: type revolute, parent Torso, child j0, origin xyz=0 -0.36461291070214186 1.6887325832692073 rpy=0 0 1, axis 1 0 0, limit lower=-3.14159 upper=3.14159 effort=0.0 velocity=0.0
- added joint Torso_k0: type revolute, parent Torso, child k0, origin xyz=0 0 2.251643444358943 rpy=0 0 1, axis 1 0 0, limit lower=-3.14159 upper=3.14159 effort=0.0 velocity=0.0
- added joint i0_i1: type revolute, parent i0, child i1, origin xyz=0 0.8671980434301998 0 rpy=1 0 0, axis 1 0 0, limit lower=-3.14159 upper=3.14159 effort=0.0 velocity=0.0
- added joint j0_j1: type revolute, parent j0, child j1, origin xyz=0 -0.7392876657518792 0 rpy=1 0 0, axis 1 0 0, limit lower=-3.14159 upper=3.14159 effort=0.0 velocity=0.0
- added joint k0_k1: type revolute, parent k0, child k1, origin xyz=0 0 0.4752483356864448 rpy=1 0 0, axis 1 0 0, limit lower=-3.14159 upper=3.14159 effort=0.0 velocity=0.0
- joint Torso_i0: origin xyz=0 0.21769121565976388 0.6147810551789473 rpy=0 1 0 -> xyz=0 0.36461291070214186 1.6887325832692073 rpy=0 0 0

File: body9.urdf (robot description, URDF)
Before this commit: robot robot, 5 links, 4 joints
Links:
- removed link i2
- added link j0, mass 1; collision box size=0.5756628666602228 0.7392876657518792 0.31631609887733225; visual box size=0.5756628666602228 0.7392876657518792 0.31631609887733225
- added link j1, mass 1; collision box size=0.995159994125997 0.6275858017941741 0.6060072164258576; visual box size=0.995159994125997 0.6275858017941741 0.6060072164258576
- added link k1, mass 1; collision box size=0.8203947820122648 0.4270699520020683 0.3215233129628592; visual box size=0.8203947820122648 0.4270699520020683 0.3215233129628592
- link Torso: geometry collision box size=0.7270228655515488 0.7292258214042837 1.1258217221794715; visual box size=0.7270228655515488 0.7292258214042837 1.1258217221794715
- link i0: geometry collision box size=0.2244946194776435 0.8671980434301998 0.44899747028739334; visual box size=0.2244946194776435 0.8671980434301998 0.44899747028739334
- link i1: geometry collision box size=0.8310824608995113 0.24893751158378974 0.6868873738781187; visual box size=0.8310824608995113 0.24893751158378974 0.6868873738781187
- link k0: geometry collision box size=0.3603192808325041 0.8881112222223901 0.4752483356864448; visual box size=0.3603192808325041 0.8881112222223901 0.4752483356864448
Joints:
- removed joint i1_i2
- added joint Torso_j0: type revolute, parent Torso, child j0, origin xyz=0 -0.36461291070214186 1.6887325832692073 rpy=0 0 1, axis 1 0 0, limit lower=-3.14159 upper=3.14159 effort=0.0 velocity=0.0
- added joint j0_j1: type revolute, parent j0, child j1, origin xyz=0 -0.7392876657518792 0 rpy=1 0 0, axis 1 0 0, limit lower=-3.14159 upper=3.14159 effort=0.0 velocity=0.0
- added joint k0_k1: type revolute, parent k0, child k1, origin xyz=0 0 0.4752483356864448 rpy=1 0 0, axis 1 0 0, limit lower=-3.14159 upper=3.14159 effort=0.0 velocity=0.0
- joint Torso_i0: origin xyz=0 0.38130821916128144 0.6953900136654471 rpy=0 1 0 -> xyz=0 0.36461291070214186 1.6887325832692073 rpy=0 1 0
- joint Torso_k0: origin xyz=0 0 0.9271866848872627 rpy=0 0 1 -> xyz=0 0 2.251643444358943 rpy=0 0 1
- joint i0_i1: origin xyz=0 0.3015601719956716 0 rpy=1 0 0 -> xyz=0 0.8671980434301998 0 rpy=1 0 0
