Commit message: done

File: body0.urdf (robot description, URDF)
Before this commit: robot robot, 7 links, 6 joints
Links:
- link Torso: geometry collision box size=1.0757034547679152 0.9626053081426966 0.6692813408980722; visual box size=1.0757034547679152 0.9626053081426966 0.6692813408980722
- link i0: geometry collision box size=0.9997766428452508 0.5543962563968308 0.9157931369904639; visual box size=0.9997766428452508 0.5543962563968308 0.9157931369904639
- link i1: geometry collision box size=0.6939725120920583 0.3365239953779773 0.501835926437016; visual box size=0.6939725120920583 0.3365239953779773 0.501835926437016
- link j0: geometry collision box size=0.43532946337780365 0.9370081597628903 0.520541839911537; visual box size=0.43532946337780365 0.9370081597628903 0.520541839911537
- link j1: geometry collision box size=0.526295212527793 0.6786671351873379 0.6437876151488082; visual box size=0.526295212527793 0.6786671351873379 0.6437876151488082
- link k0: geometry collision box size=0.8940809661088207 0.6202708299025574 0.9394122376082263; visual box size=0.8940809661088207 0.6202708299025574 0.9394122376082263
- link k1: geometry collision box size=0.6347262754269247 0.9368920826888067 0.7478614554556864; visual box size=0.6347262754269247 0.9368920826888067 0.7478614554556864
Joints:
- joint Torso_i0: origin xyz=0 0.36461291070214186 1.6887325832692073 rpy=1 0 0 -> xyz=0 0.4813026540713483 1.0039220113471083 rpy=0 1 0
- joint Torso_j0: origin xyz=0 -0.36461291070214186 1.6887325832692073 rpy=0 0 1 -> xyz=0 -0.4813026540713483 1.0039220113471083 rpy=0 0 1
- joint Torso_k0: origin xyz=0 0 2.251643444358943 rpy=0 0 1 -> xyz=0 0 1.3385626817961445 rpy=0 0 1
- joint i0_i1: origin xyz=0 0.8671980434301998 0 rpy=1 0 0 -> xyz=0.9997766428452508 0.5543962563968308 0 rpy=1 0 0
- joint j0_j1: origin xyz=0 -0.7392876657518792 0 rpy=1 0 0 -> xyz=0 -0.9370081597628903 0 rpy=1 0 0
- joint k0_k1: origin xyz=0 0 0.4752483356864448 rpy=1 0 0 -> xyz=0 0 0.9394122376082263 rpy=1 0 0

File: body1.urdf (robot description, URDF)
Before this commit: robot robot, 7 links, 6 joints
Links:
- link Torso: geometry collision box size=1.0757034547679152 0.9626053081426966 0.6692813408980722; visual box size=1.0757034547679152 0.9626053081426966 0.6692813408980722
- link i0: geometry collision box size=0.9997766428452508 0.5543962563968308 0.9157931369904639; visual box size=0.9997766428452508 0.5543962563968308 0.9157931369904639
- link i1: geometry collision box size=0.6939725120920583 0.3365239953779773 0.501835926437016; visual box size=0.6939725120920583 0.3365239953779773 0.501835926437016
- link j0: geometry collision box size=0.43532946337780365 0.9370081597628903 0.520541839911537; visual box size=0.43532946337780365 0.9370081597628903 0.520541839911537
- link j1: geometry collision box size=0.526295212527793 0.6786671351873379 0.6437876151488082; visual box size=0.526295212527793 0.6786671351873379 0.6437876151488082
- link k0: geometry collision box size=0.8940809661088207 0.6202708299025574 0.9394122376082263; visual box size=0.8940809661088207 0.6202708299025574 0.9394122376082263
- link k1: geometry collision box size=0.6347262754269247 0.9368920826888067 0.7478614554556864; visual box size=0.6347262754269247 0.9368920826888067 0.7478614554556864
Joints:
- joint Torso_i0: origin xyz=0 0.36461291070214186 1.6887325832692073 rpy=0 0 1 -> xyz=0 0.4813026540713483 1.0039220113471083 rpy=0 1 0
- joint Torso_j0: origin xyz=0 -0.36461291070214186 1.6887325832692073 rpy=0 0 1 -> xyz=0 -0.4813026540713483 1.0039220113471083 rpy=0 0 1
- joint Torso_k0: origin xyz=0 0 2.251643444358943 rpy=0 0 1 -> xyz=0 0 1.3385626817961445 rpy=0 0 1
- joint i0_i1: origin xyz=0 0.8671980434301998 0 rpy=1 0 0 -> xyz=0.9997766428452508 0.5543962563968308 0 rpy=1 0 0
- joint j0_j1: origin xyz=0 -0.7392876657518792 0 rpy=1 0 0 -> xyz=0 -0.9370081597628903 0 rpy=1 0 0
- joint k0_k1: origin xyz=0 0 0.4752483356864448 rpy=1 0 0 -> xyz=0 0 0.9394122376082263 rpy=1 0 0

File: body10.urdf (robot description, URDF)
Before this commit: robot robot, 7 links, 6 joints
Links:
- link Torso: geometry collision box size=1.0757034547679152 0.9626053081426966 0.6692813408980722; visual box size=1.0757034547679152 0.9626053081426966 0.6692813408980722
- link i0: geometry collision box size=0.9997766428452508 0.5543962563968308 0.9157931369904639; visual box size=0.9997766428452508 0.5543962563968308 0.9157931369904639
- link i1: geometry collision box size=0.6939725120920583 0.3365239953779773 0.501835926437016; visual box size=0.6939725120920583 0.3365239953779773 0.501835926437016
- link j0: geometry collision box size=0.43532946337780365 0.9370081597628903 0.520541839911537; visual box size=0.43532946337780365 0.9370081597628903 0.520541839911537
- link j1: geometry collision box size=0.526295212527793 0.6786671351873379 0.6437876151488082; visual box size=0.526295212527793 0.6786671351873379 0.6437876151488082
- link k0: geometry collision box size=0.8940809661088207 0.6202708299025574 0.9394122376082263; visual box size=0.8940809661088207 0.6202708299025574 0.9394122376082263
- link k1: geometry collision box size=0.6347262754269247 0.9368920826888067 0.7478614554556864; visual box size=0.6347262754269247 0.9368920826888067 0.7478614554556864
Joints:
- joint Torso_i0: origin xyz=0 0.36461291070214186 1.6887325832692073 rpy=1 0 0 -> xyz=0 0.4813026540713483 1.0039220113471083 rpy=1 0 0
- joint Torso_j0: origin xyz=0 -0.36461291070214186 1.6887325832692073 rpy=0 0 1 -> xyz=0 -0.4813026540713483 1.0039220113471083 rpy=0 0 1
- joint Torso_k0: origin xyz=0 0 2.251643444358943 rpy=0 0 1 -> xyz=0 0 1.3385626817961445 rpy=0 0 1
- joint i0_i1: origin xyz=0 0.8671980434301998 0 rpy=1 0 0 -> xyz=0.9997766428452508 0.5543962563968308 0 rpy=1 0 0
- joint j0_j1: origin xyz=0 -0.7392876657518792 0 rpy=1 0 0 -> xyz=0 -0.9370081597628903 0 rpy=1 0 0
- joint k0_k1: origin xyz=0 0 0.4752483356864448 rpy=1 0 0 -> xyz=0 0 0.9394122376082263 rpy=1 0 0

File: body2.urdf (robot description, URDF)
Before this commit: robot robot, 7 links, 6 joints
Links:
- link Torso: geometry collision box size=1.0757034547679152 0.9626053081426966 0.6692813408980722; visual box size=1.0757034547679152 0.9626053081426966 0.6692813408980722
- link i0: geometry collision box size=0.9997766428452508 0.5543962563968308 0.9157931369904639; visual box size=0.9997766428452508 0.5543962563968308 0.9157931369904639
- link i1: geometry collision box size=0.6939725120920583 0.3365239953779773 0.501835926437016; visual box size=0.6939725120920583 0.3365239953779773 0.501835926437016
- link j0: geometry collision box size=0.43532946337780365 0.9370081597628903 0.520541839911537; visual box size=0.43532946337780365 0.9370081597628903 0.520541839911537
- link j1: geometry collision box size=0.526295212527793 0.6786671351873379 0.6437876151488082; visual box size=0.526295212527793 0.6786671351873379 0.6437876151488082
- link k0: geometry collision box size=0.8940809661088207 0.6202708299025574 0.9394122376082263; visual box size=0.8940809661088207 0.6202708299025574 0.9394122376082263
- link k1: geometry collision box size=0.6347262754269247 0.9368920826888067 0.7478614554556864; visual box size=0.6347262754269247 0.9368920826888067 0.7478614554556864
Joints:
- joint Torso_i0: origin xyz=0 0.36461291070214186 1.6887325832692073 rpy=0 1 0 -> xyz=0 0.4813026540713483 1.0039220113471083 rpy=0 0 0
- joint Torso_j0: origin xyz=0 -0.36461291070214186 1.6887325832692073 rpy=0 0 1 -> xyz=0 -0.4813026540713483 1.0039220113471083 rpy=0 0 1
- joint Torso_k0: origin xyz=0 0 2.251643444358943 rpy=0 0 1 -> xyz=0 0 1.3385626817961445 rpy=0 0 1
- joint i0_i1: origin xyz=0 0.8671980434301998 0 rpy=1 0 0 -> xyz=0.9997766428452508 0.5543962563968308 0 rpy=1 0 0
- joint j0_j1: origin xyz=0 -0.7392876657518792 0 rpy=1 0 0 -> xyz=0 -0.9370081597628903 0 rpy=1 0 0
- joint k0_k1: origin xyz=0 0 0.4752483356864448 rpy=1 0 0 -> xyz=0 0 0.9394122376082263 rpy=1 0 0

File: body3.urdf (robot description, URDF)
Before this commit: robot robot, 7 links, 6 joints
Links:
- link Torso: geometry collision box size=1.0757034547679152 0.9626053081426966 0.6692813408980722; visual box size=1.0757034547679152 0.9626053081426966 0.6692813408980722
- link i0: geometry collision box size=0.9997766428452508 0.5543962563968308 0.9157931369904639; visual box size=0.9997766428452508 0.5543962563968308 0.9157931369904639
- link i1: geometry collision box size=0.6939725120920583 0.3365239953779773 0.501835926437016; visual box size=0.6939725120920583 0.3365239953779773 0.501835926437016
- link j0: geometry collision box size=0.43532946337780365 0.9370081597628903 0.520541839911537; visual box size=0.43532946337780365 0.9370081597628903 0.520541839911537
- link j1: geometry collision box size=0.526295212527793 0.6786671351873379 0.6437876151488082; visual box size=0.526295212527793 0.6786671351873379 0.6437876151488082
- link k0: geometry collision box size=0.8940809661088207 0.6202708299025574 0.9394122376082263; visual box size=0.8940809661088207 0.6202708299025574 0.9394122376082263
- link k1: geometry collision box size=0.6347262754269247 0.9368920826888067 0.7478614554556864; visual box size=0.6347262754269247 0.9368920826888067 0.7478614554556864
Joints:
- joint Torso_i0: origin xyz=0 0.36461291070214186 1.6887325832692073 rpy=1 0 0 -> xyz=0 0.4813026540713483 1.0039220113471083 rpy=1 0 0
- joint Torso_j0: origin xyz=0 -0.36461291070214186 1.6887325832692073 rpy=0 0 1 -> xyz=0 -0.4813026540713483 1.0039220113471083 rpy=0 0 1
- joint Torso_k0: origin xyz=0 0 2.251643444358943 rpy=0 0 1 -> xyz=0 0 1.3385626817961445 rpy=0 0 1
- joint i0_i1: origin xyz=0 0.8671980434301998 0 rpy=1 0 0 -> xyz=0.9997766428452508 0.5543962563968308 0 rpy=1 0 0
- joint j0_j1: origin xyz=0 -0.7392876657518792 0 rpy=1 0 0 -> xyz=0 -0.9370081597628903 0 rpy=1 0 0
- joint k0_k1: origin xyz=0 0 0.4752483356864448 rpy=1 0 0 -> xyz=0 0 0.9394122376082263 rpy=1 0 0

File: body4.urdf (robot description, URDF)
Before this commit: robot robot, 7 links, 6 joints
Links:
- link Torso: geometry collision box size=1.0757034547679152 0.9626053081426966 0.6692813408980722; visual box size=1.0757034547679152 0.9626053081426966 0.6692813408980722
- link i0: geometry collision box size=0.9997766428452508 0.5543962563968308 0.9157931369904639; visual box size=0.9997766428452508 0.5543962563968308 0.9157931369904639
- link i1: geometry collision box size=0.6939725120920583 0.3365239953779773 0.501835926437016; visual box size=0.6939725120920583 0.3365239953779773 0.501835926437016
- link j0: geometry collision box size=0.43532946337780365 0.9370081597628903 0.520541839911537; visual box size=0.43532946337780365 0.9370081597628903 0.520541839911537
- link j1: geometry collision box size=0.526295212527793 0.6786671351873379 0.6437876151488082; visual box size=0.526295212527793 0.6786671351873379 0.6437876151488082
- link k0: geometry collision box size=0.8940809661088207 0.6202708299025574 0.9394122376082263; visual box size=0.8940809661088207 0.6202708299025574 0.9394122376082263
- link k1: geometry collision box size=0.6347262754269247 0.9368920826888067 0.7478614554556864; visual box size=0.6347262754269247 0.9368920826888067 0.7478614554556864
Joints:
- joint Torso_i0: origin xyz=0 0.36461291070214186 1.6887325832692073 rpy=0 0 0 -> xyz=0 0.4813026540713483 1.0039220113471083 rpy=0 0 0
- joint Torso_j0: origin xyz=0 -0.36461291070214186 1.6887325832692073 rpy=0 0 1 -> xyz=0 -0.4813026540713483 1.0039220113471083 rpy=0 0 1
- joint Torso_k0: origin xyz=0 0 2.251643444358943 rpy=0 0 1 -> xyz=0 0 1.3385626817961445 rpy=0 0 1
- joint i0_i1: origin xyz=0 0.8671980434301998 0 rpy=1 0 0 -> xyz=0.9997766428452508 0.5543962563968308 0 rpy=1 0 0
- joint j0_j1: origin xyz=0 -0.7392876657518792 0 rpy=1 0 0 -> xyz=0 -0.9370081597628903 0 rpy=1 0 0
- joint k0_k1: origin xyz=0 0 0.4752483356864448 rpy=1 0 0 -> xyz=0 0 0.9394122376082263 rpy=1 0 0

File: body5.urdf (robot description, URDF)
Before this commit: robot robot, 7 links, 6 joints
Links:
- link Torso: geometry collision box size=1.0757034547679152 0.9626053081426966 0.6692813408980722; visual box size=1.0757034547679152 0.9626053081426966 0.6692813408980722
- link i0: geometry collision box size=0.9997766428452508 0.5543962563968308 0.9157931369904639; visual box size=0.9997766428452508 0.5543962563968308 0.9157931369904639
- link i1: geometry collision box size=0.6939725120920583 0.3365239953779773 0.501835926437016; visual box size=0.6939725120920583 0.3365239953779773 0.501835926437016
- link j0: geometry collision box size=0.43532946337780365 0.9370081597628903 0.520541839911537; visual box size=0.43532946337780365 0.9370081597628903 0.520541839911537
- link j1: geometry collision box size=0.526295212527793 0.6786671351873379 0.6437876151488082; visual box size=0.526295212527793 0.6786671351873379 0.6437876151488082
- link k0: geometry collision box size=0.8940809661088207 0.6202708299025574 0.9394122376082263; visual box size=0.8940809661088207 0.6202708299025574 0.9394122376082263
- link k1: geometry collision box size=0.6347262754269247 0.9368920826888067 0.7478614554556864; visual box size=0.6347262754269247 0.9368920826888067 0.7478614554556864
Joints:
- joint Torso_i0: origin xyz=0 0.36461291070214186 1.6887325832692073 rpy=0 1 0 -> xyz=0 0.4813026540713483 1.0039220113471083 rpy=1 0 0
- joint Torso_j0: origin xyz=0 -0.36461291070214186 1.6887325832692073 rpy=0 0 1 -> xyz=0 -0.4813026540713483 1.0039220113471083 rpy=0 0 1
- joint Torso_k0: origin xyz=0 0 2.251643444358943 rpy=0 0 1 -> xyz=0 0 1.3385626817961445 rpy=0 0 1
- joint i0_i1: origin xyz=0 0.8671980434301998 0 rpy=1 0 0 -> xyz=0.9997766428452508 0.5543962563968308 0 rpy=1 0 0
- joint j0_j1: origin xyz=0 -0.7392876657518792 0 rpy=1 0 0 -> xyz=0 -0.9370081597628903 0 rpy=1 0 0
- joint k0_k1: origin xyz=0 0 0.4752483356864448 rpy=1 0 0 -> xyz=0 0 0.9394122376082263 rpy=1 0 0

File: body6.urdf (robot description, URDF)
Before this commit: robot robot, 7 links, 6 joints
Links:
- link Torso: geometry collision box size=1.0757034547679152 0.9626053081426966 0.6692813408980722; visual box size=1.0757034547679152 0.9626053081426966 0.6692813408980722
- link i0: geometry collision box size=0.9997766428452508 0.5543962563968308 0.9157931369904639; visual box size=0.9997766428452508 0.5543962563968308 0.9157931369904639
- link i1: geometry collision box size=0.6939725120920583 0.3365239953779773 0.501835926437016; visual box size=0.6939725120920583 0.3365239953779773 0.501835926437016
- link j0: geometry collision box size=0.43532946337780365 0.9370081597628903 0.520541839911537; visual box size=0.43532946337780365 0.9370081597628903 0.520541839911537
- link j1: geometry collision box size=0.526295212527793 0.6786671351873379 0.6437876151488082; visual box size=0.526295212527793 0.6786671351873379 0.6437876151488082
- link k0: geometry collision box size=0.8940809661088207 0.6202708299025574 0.9394122376082263; visual box size=0.8940809661088207 0.6202708299025574 0.9394122376082263
- link k1: geometry collision box size=0.6347262754269247 0.9368920826888067 0.7478614554556864; visual box size=0.6347262754269247 0.9368920826888067 0.7478614554556864
Joints:
- joint Torso_i0: origin xyz=0 0.36461291070214186 1.6887325832692073 rpy=0 1 0 -> xyz=0 0.4813026540713483 1.0039220113471083 rpy=0 0 0
- joint Torso_j0: origin xyz=0 -0.36461291070214186 1.6887325832692073 rpy=0 0 1 -> xyz=0 -0.4813026540713483 1.0039220113471083 rpy=0 0 1
- joint Torso_k0: origin xyz=0 0 2.251643444358943 rpy=0 0 1 -> xyz=0 0 1.3385626817961445 rpy=0 0 1
- joint i0_i1: origin xyz=0 0.8671980434301998 0 rpy=1 0 0 -> xyz=0.9997766428452508 0.5543962563968308 0 rpy=1 0 0
- joint j0_j1: origin xyz=0 -0.7392876657518792 0 rpy=1 0 0 -> xyz=0 -0.9370081597628903 0 rpy=1 0 0
- joint k0_k1: origin xyz=0 0 0.4752483356864448 rpy=1 0 0 -> xyz=0 0 0.9394122376082263 rpy=1 0 0

File: body7.urdf (robot description, URDF)
Before this commit: robot robot, 7 links, 6 joints
Links:
- link Torso: geometry collision box size=1.0757034547679152 0.9626053081426966 0.6692813408980722; visual box size=1.0757034547679152 0.9626053081426966 0.6692813408980722
- link i0: geometry collision box size=0.9997766428452508 0.5543962563968308 0.9157931369904639; visual box size=0.9997766428452508 0.5543962563968308 0.9157931369904639
- link i1: geometry collision box size=0.6939725120920583 0.3365239953779773 0.501835926437016; visual box size=0.6939725120920583 0.3365239953779773 0.501835926437016
- link j0: geometry collision box size=0.43532946337780365 0.9370081597628903 0.520541839911537; visual box size=0.43532946337780365 0.9370081597628903 0.520541839911537
- link j1: geometry collision box size=0.526295212527793 0.6786671351873379 0.6437876151488082; visual box size=0.526295212527793 0.6786671351873379 0.6437876151488082
- link k0: geometry collision box size=0.8940809661088207 0.6202708299025574 0.9394122376082263; visual box size=0.8940809661088207 0.6202708299025574 0.9394122376082263
- link k1: geometry collision box size=0.6347262754269247 0.9368920826888067 0.7478614554556864; visual box size=0.6347262754269247 0.9368920826888067 0.7478614554556864
Joints:
- joint Torso_i0: origin xyz=0 0.36461291070214186 1.6887325832692073 rpy=1 0 0 -> xyz=0 0.4813026540713483 1.0039220113471083 rpy=0 1 0
- joint Torso_j0: origin xyz=0 -0.36461291070214186 1.6887325832692073 rpy=0 0 1 -> xyz=0 -0.4813026540713483 1.0039220113471083 rpy=0 0 1
- joint Torso_k0: origin xyz=0 0 2.251643444358943 rpy=0 0 1 -> xyz=0 0 1.3385626817961445 rpy=0 0 1
- joint i0_i1: origin xyz=0 0.8671980434301998 0 rpy=1 0 0 -> xyz=0.9997766428452508 0.5543962563968308 0 rpy=1 0 0
- joint j0_j1: origin xyz=0 -0.7392876657518792 0 rpy=1 0 0 -> xyz=0 -0.9370081597628903 0 rpy=1 0 0
- joint k0_k1: origin xyz=0 0 0.4752483356864448 rpy=1 0 0 -> xyz=0 0 0.9394122376082263 rpy=1 0 0

File: body8.urdf (robot description, URDF)
Before this commit: robot robot, 7 links, 6 joints
Links:
- link Torso: geometry collision box size=1.0757034547679152 0.9626053081426966 0.6692813408980722; visual box size=1.0757034547679152 0.9626053081426966 0.6692813408980722
- link i0: geometry collision box size=0.9997766428452508 0.5543962563968308 0.9157931369904639; visual box size=0.9997766428452508 0.5543962563968308 0.9157931369904639
- link i1: geometry collision box size=0.6939725120920583 0.3365239953779773 0.501835926437016; visual box size=0.6939725120920583 0.3365239953779773 0.501835926437016
- link j0: geometry collision box size=0.43532946337780365 0.9370081597628903 0.520541839911537; visual box size=0.43532946337780365 0.9370081597628903 0.520541839911537
- link j1: geometry collision box size=0.526295212527793 0.6786671351873379 0.6437876151488082; visual box size=0.526295212527793 0.6786671351873379 0.6437876151488082
- link k0: geometry collision box size=0.8940809661088207 0.6202708299025574 0.9394122376082263; visual box size=0.8940809661088207 0.6202708299025574 0.9394122376082263
- link k1: geometry collision box size=0.6347262754269247 0.9368920826888067 0.7478614554556864; visual box size=0.6347262754269247 0.9368920826888067 0.7478614554556864
Joints:
- joint Torso_i0: origin xyz=0 0.36461291070214186 1.6887325832692073 rpy=0 0 0 -> xyz=0 0.4813026540713483 1.0039220113471083 rpy=1 0 0
- joint Torso_j0: origin xyz=0 -0.36461291070214186 1.6887325832692073 rpy=0 0 1 -> xyz=0 -0.4813026540713483 1.0039220113471083 rpy=0 0 1
- joint Torso_k0: origin xyz=0 0 2.251643444358943 rpy=0 0 1 -> xyz=0 0 1.3385626817961445 rpy=0 0 1
- joint i0_i1: origin xyz=0 0.8671980434301998 0 rpy=1 0 0 -> xyz=0.9997766428452508 0.5543962563968308 0 rpy=1 0 0
- joint j0_j1: origin xyz=0 -0.7392876657518792 0 rpy=1 0 0 -> xyz=0 -0.9370081597628903 0 rpy=1 0 0
- joint k0_k1: origin xyz=0 0 0.4752483356864448 rpy=1 0 0 -> xyz=0 0 0.9394122376082263 rpy=1 0 0

File: body9.urdf (robot description, URDF)
Before this commit: robot robot, 7 links, 6 joints
Links:
- link Torso: geometry collision box size=1.0757034547679152 0.9626053081426966 0.6692813408980722; visual box size=1.0757034547679152 0.9626053081426966 0.6692813408980722
- link i0: geometry collision box size=0.9997766428452508 0.5543962563968308 0.9157931369904639; visual box size=0.9997766428452508 0.5543962563968308 0.9157931369904639
- link i1: geometry collision box size=0.6939725120920583 0.3365239953779773 0.501835926437016; visual box size=0.6939725120920583 0.3365239953779773 0.501835926437016
- link j0: geometry collision box size=0.43532946337780365 0.9370081597628903 0.520541839911537; visual box size=0.43532946337780365 0.9370081597628903 0.520541839911537
- link j1: geometry collision box size=0.526295212527793 0.6786671351873379 0.6437876151488082; visual box size=0.526295212527793 0.6786671351873379 0.6437876151488082
- link k0: geometry collision box size=0.8940809661088207 0.6202708299025574 0.9394122376082263; visual box size=0.8940809661088207 0.6202708299025574 0.9394122376082263
- link k1: geometry collision box size=0.6347262754269247 0.9368920826888067 0.7478614554556864; visual box size=0.6347262754269247 0.9368920826888067 0.7478614554556864
Joints:
- joint Torso_i0: origin xyz=0 0.36461291070214186 1.6887325832692073 rpy=0 1 0 -> xyz=0 0.4813026540713483 1.0039220113471083 rpy=0 1 0
- joint Torso_j0: origin xyz=0 -0.36461291070214186 1.6887325832692073 rpy=0 0 1 -> xyz=0 -0.4813026540713483 1.0039220113471083 rpy=0 0 1
- joint Torso_k0: origin xyz=0 0 2.251643444358943 rpy=0 0 1 -> xyz=0 0 1.3385626817961445 rpy=0 0 1
- joint i0_i1: origin xyz=0 0.8671980434301998 0 rpy=1 0 0 -> xyz=0.9997766428452508 0.5543962563968308 0 rpy=1 0 0
- joint j0_j1: origin xyz=0 -0.7392876657518792 0 rpy=1 0 0 -> xyz=0 -0.9370081597628903 0 rpy=1 0 0
- joint k0_k1: origin xyz=0 0 0.4752483356864448 rpy=1 0 0 -> xyz=0 0 0.9394122376082263 rpy=1 0 0
